File: pisxme/reva-clean/ACREAGE_CANDIDATE.kicad_pcb (KiCad board)
At the start: 6 copper layers, 300 x 180 mm, 20 parts, among them J1 74221-101LF, J2 A70-112-331N126, J3 JAE SM3ZS067U410ABR1000 B-key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, J4 Amphenol 10171746-00021LF USB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, U1 LM74700QDBVRQ1, U2 LM74700QDBVRQ1, U3 TPSM63606RDLR, U4 TPSM63606RDLR, U5 TPSM63606RDLR, U6 TPD4E004DRYR, U7 TUSB9261IPVP, U8 Texas_DRT_3, U9 TPD4E004DRYR

Commit message: promote native CM5 and materialize clean candidate
Parts:
- removed REF**: Raspberry-Pi-5-Compute-Module, PiSXMeRevAClean_Raspberry_Pi_5_Compute_Module
- added J5: 0039300020, Molex_0039300020_5569_2P_RA, F.Cu at (12.0, 25.0)
- added J6: 0039300020, Molex_0039300020_5569_2P_RA, F.Cu at (12.0, 45.0)
- added J7: Raspberry-Pi-5-Compute-Module, PiSXMeRevAClean_Raspberry_Pi_5_Compute_Module, B.Cu at (35.0, 130.0)

Commit message: close phase5 power architecture gate
Parts:
- added C14: , C_1206_3216Metric, F.Cu at (70.0, 120.0)
- added C15: , C_1206_3216Metric, F.Cu at (78.0, 120.0)
- added C16: , C_1210_3225Metric, F.Cu at (86.0, 120.0)
- added C17: , C_1210_3225Metric, F.Cu at (94.0, 120.0)
- added C18: C_0805_2012Metric, C_0805_2012Metric, F.Cu at (102.0, 120.0)
- added C19: , C_1210_3225Metric, F.Cu at (110.0, 120.0)
- added C23: , C_1206_3216Metric, F.Cu at (70.0, 170.0)
- added C24: C_0805_2012Metric, C_0805_2012Metric, F.Cu at (78.0, 170.0)
- added C25: , C_1206_3216Metric, F.Cu at (86.0, 170.0)
- added C26: , C_1210_3225Metric, F.Cu at (150.0, 150.0)
- added C27: , C_1210_3225Metric, F.Cu at (158.0, 150.0)
- added C28: , C_1210_3225Metric, F.Cu at (166.0, 150.0)
- added C29: , C_1210_3225Metric, F.Cu at (174.0, 150.0)
- added C3: C_0603_1608Metric, C_0603_1608Metric, F.Cu at (110.0, 55.0)
- added C30: , C_1210_3225Metric, F.Cu at (182.0, 150.0)
- added C31: , C_1210_3225Metric, F.Cu at (190.0, 150.0)
- added C32: , C_1210_3225Metric, F.Cu at (198.0, 150.0)
- added C33: , C_1210_3225Metric, F.Cu at (206.0, 150.0)
- added C34: , C_1210_3225Metric, F.Cu at (150.0, 158.0)
- added C35: , C_1210_3225Metric, F.Cu at (158.0, 158.0)
- added C36: , C_1210_3225Metric, F.Cu at (166.0, 158.0)
- added C37: , C_1210_3225Metric, F.Cu at (174.0, 158.0)
- added C38: , C_1210_3225Metric, F.Cu at (182.0, 158.0)
- added C39: , C_1210_3225Metric, F.Cu at (190.0, 158.0)
- added C4: C_0603_1608Metric, C_0603_1608Metric, F.Cu at (110.0, 95.0)
- added C40: , C_1210_3225Metric, F.Cu at (198.0, 158.0)
- added C41: , C_1210_3225Metric, F.Cu at (206.0, 158.0)
- added C5: , C_1206_3216Metric, F.Cu at (70.0, 70.0)
- added C6: , C_1206_3216Metric, F.Cu at (78.0, 70.0)
- added C7: , C_1210_3225Metric, F.Cu at (86.0, 70.0)
- added C8: , C_1210_3225Metric, F.Cu at (94.0, 70.0)
- added C9: C_0805_2012Metric, C_0805_2012Metric, F.Cu at (102.0, 70.0)
- added D1: SMBJ18A, TVS_SMBJ18A_DO214AA, F.Cu at (110.0, 32.0)
- added D2: SMBJ18A, TVS_SMBJ18A_DO214AA, F.Cu at (110.0, 72.0)
- added F1: 178.6165.0001, ATO_FuseHolder_17861650001, F.Cu at (90.0, 40.0)
- added F2: 178.6165.0001, ATO_FuseHolder_17861650001, F.Cu at (90.0, 80.0)
- added Q1: CSD19536KCS, CSD19536KCS_TO220, F.Cu at (130.0, 40.0)
- added Q2: CSD19536KCS, CSD19536KCS_TO220, F.Cu at (130.0, 80.0)
- added R11: R_0402_1005Metric, R_0402_1005Metric, F.Cu at (70.0, 132.0)
- added R12: R_0402_1005Metric, R_0402_1005Metric, F.Cu at (78.0, 132.0)
- added R13: R_0402_1005Metric, R_0402_1005Metric, F.Cu at (86.0, 132.0)
- added R14: R_0402_1005Metric, R_0402_1005Metric, F.Cu at (94.0, 132.0)
- added R19: R_0402_1005Metric, R_0402_1005Metric, F.Cu at (94.0, 170.0)
- added R20: R_0402_1005Metric, R_0402_1005Metric, F.Cu at (102.0, 170.0)
- added R21: R_0402_1005Metric, R_0402_1005Metric, F.Cu at (110.0, 170.0)
- added R22: R_0402_1005Metric, R_0402_1005Metric, F.Cu at (118.0, 170.0)
- added R3: R_0402_1005Metric, R_0402_1005Metric, F.Cu at (70.0, 82.0)
- added R4: R_0402_1005Metric, R_0402_1005Metric, F.Cu at (78.0, 82.0)
- added R5: R_0402_1005Metric, R_0402_1005Metric, F.Cu at (86.0, 82.0)
- added R6: R_0402_1005Metric, R_0402_1005Metric, F.Cu at (94.0, 82.0)
Connections:
- J1 pad A3: /V100_PCIE/V100_POWER_12V -> 12V_PROTECTED
- J5 pad 1: Net-(J5-12V) -> /POWER_INPUT/12V_IN_A
- J5 pad 2: Net-(J5-GND) -> /POWER_INPUT/POWER_GND
- J6 pad 1: Net-(J5-12V) -> /POWER_INPUT/12V_IN_B
- J6 pad 2: Net-(J5-GND) -> /POWER_INPUT/POWER_GND
- U1 pad 1: /POWER_INPUT/POWER_PG_FAULT -> /POWER_INPUT/VCAP_A
- U1 pad 3: /POWER_INPUT/12V_PROTECTED -> /POWER_INPUT/12V_IN_A
- U1 pad 4: /POWER_INPUT/12V_IN_A -> 12V_PROTECTED
- U1 pad 5: (no net) -> /POWER_INPUT/GATE_A
- U1 pad 6: (no net) -> /POWER_INPUT/FUSED_12V_A
- U2 pad 1: /POWER_INPUT/POWER_PG_FAULT -> /POWER_INPUT/VCAP_B
- U2 pad 3: /POWER_INPUT/12V_PROTECTED -> /POWER_INPUT/12V_IN_B
- U2 pad 4: /POWER_INPUT/12V_IN_A -> 12V_PROTECTED
- U2 pad 5: (no net) -> /POWER_INPUT/GATE_B
- U2 pad 6: (no net) -> /POWER_INPUT/FUSED_12V_B
- U3 pad 1: /REGULATORS/BRIDGE_ENABLE -> /REGULATORS/12V_PROTECTED
- U3 pad 10: (no net) -> /REGULATORS/FB_CM5_5V
- U3 pad 11: (no net) -> /REGULATORS/POWER_GND
- U3 pad 12: (no net) -> /REGULATORS/RT_CM5_5V
- U3 pad 13: (no net) -> /REGULATORS/PG_CM5_5V
- U3 pad 14: (no net) -> /REGULATORS/12V_PROTECTED
- U3 pad 15: (no net) -> /REGULATORS/NC
- U3 pad 16: (no net) -> /REGULATORS/12V_PROTECTED
- U3 pad 17: (no net) -> /REGULATORS/POWER_GND
- U3 pad 18: (no net) -> /REGULATORS/POWER_GND
- U3 pad 19: (no net) -> /REGULATORS/POWER_GND
- U3 pad 2: /REGULATORS/POWER_GND -> /REGULATORS/SW_CM5_5V
- U3 pad 20: (no net) -> /REGULATORS/POWER_GND
- U3 pad 3: /REGULATORS/BRIDGE_1V1 -> /REGULATORS/CBOOT_CM5_5V
- U3 pad 4: /REGULATORS/12V_PROTECTED -> /REGULATORS/RBOOT_CM5_5V
- U3 pad 5: (no net) -> /REGULATORS/12V_PROTECTED
- U3 pad 6: (no net) -> /REGULATORS/POWER_GND
- U3 pad 7: (no net) -> /REGULATORS/VCC_INTERNAL
- U3 pad 8: (no net) -> /REGULATORS/CM5_5V
- U3 pad 9: (no net) -> /REGULATORS/CM5_5V
- U4 pad 1: /REGULATORS/BRIDGE_ENABLE -> /REGULATORS/12V_PROTECTED
- U4 pad 10: (no net) -> /REGULATORS/FB_BRIDGE_3V3
- U4 pad 11: (no net) -> /REGULATORS/POWER_GND
- U4 pad 12: (no net) -> /REGULATORS/RT_BRIDGE_3V3
- U4 pad 13: (no net) -> /REGULATORS/PG_BRIDGE_3V3
- U4 pad 14: (no net) -> /REGULATORS/12V_PROTECTED
- U4 pad 15: (no net) -> /REGULATORS/NC
- U4 pad 16: (no net) -> /REGULATORS/12V_PROTECTED
- U4 pad 17: (no net) -> /REGULATORS/POWER_GND
- U4 pad 18: (no net) -> /REGULATORS/POWER_GND
- U4 pad 19: (no net) -> /REGULATORS/POWER_GND
- U4 pad 2: /REGULATORS/POWER_GND -> /REGULATORS/SW_BRIDGE_3V3
- U4 pad 20: (no net) -> /REGULATORS/POWER_GND
- U4 pad 3: /REGULATORS/BRIDGE_1V1 -> /REGULATORS/CBOOT_BRIDGE_3V3
- U4 pad 4: /REGULATORS/12V_PROTECTED -> /REGULATORS/RBOOT_BRIDGE_3V3
- U4 pad 5: (no net) -> /REGULATORS/12V_PROTECTED
- U4 pad 6: (no net) -> /REGULATORS/POWER_GND
- U4 pad 7: (no net) -> /REGULATORS/VCC_INTERNAL
- U4 pad 8: (no net) -> /REGULATORS/BRIDGE_3V3
- U4 pad 9: (no net) -> /REGULATORS/BRIDGE_3V3
- U5 pad 1: /REGULATORS/BRIDGE_ENABLE -> /REGULATORS/12V_PROTECTED
- U5 pad 10: (no net) -> /REGULATORS/FB_BRIDGE_1V1
- U5 pad 11: (no net) -> /REGULATORS/POWER_GND
- U5 pad 12: (no net) -> /REGULATORS/RT_BRIDGE_1V1
- U5 pad 13: (no net) -> /REGULATORS/PG_BRIDGE_1V1
- U5 pad 14: (no net) -> /REGULATORS/12V_PROTECTED
- U5 pad 15: (no net) -> /REGULATORS/NC
- U5 pad 16: (no net) -> /REGULATORS/12V_PROTECTED
- U5 pad 17: (no net) -> /REGULATORS/POWER_GND
- U5 pad 18: (no net) -> /REGULATORS/POWER_GND
- U5 pad 19: (no net) -> /REGULATORS/POWER_GND
- U5 pad 2: /REGULATORS/POWER_GND -> /REGULATORS/SW_BRIDGE_1V1
- U5 pad 20: (no net) -> /REGULATORS/POWER_GND
- U5 pad 3: /REGULATORS/BRIDGE_1V1 -> /REGULATORS/CBOOT_BRIDGE_1V1
- U5 pad 4: /REGULATORS/12V_PROTECTED -> /REGULATORS/RBOOT_BRIDGE_1V1
- U5 pad 5: (no net) -> /REGULATORS/12V_PROTECTED
- U5 pad 6: (no net) -> /REGULATORS/POWER_GND
- U5 pad 7: (no net) -> /REGULATORS/VCC_INTERNAL
- U5 pad 8: (no net) -> /REGULATORS/BRIDGE_1V1
- U5 pad 9: (no net) -> /REGULATORS/BRIDGE_1V1

Commit message: fix SXM2 native mapping and power aliases
Connections:
- J1 pad A2: /V100_PCIE/V100_GND -> /V100_PCIE/V100_PER0_P
- J1 pad A21: (no net) -> /V100_PCIE/V100_GND
- J1 pad A22: (no net) -> 12V_PROTECTED
- J1 pad A23: (no net) -> 12V_PROTECTED
- J1 pad A24: (no net) -> /V100_PCIE/V100_GND
- J1 pad A25: (no net) -> 12V_PROTECTED
- J1 pad A26: (no net) -> 12V_PROTECTED
- J1 pad A27: (no net) -> /V100_PCIE/V100_GND
- J1 pad A28: (no net) -> 12V_PROTECTED
- J1 pad A29: (no net) -> 12V_PROTECTED
- J1 pad A3: 12V_PROTECTED -> /V100_PCIE/V100_PER0_N
- J1 pad A30: (no net) -> /V100_PCIE/V100_GND
- J1 pad A31: (no net) -> 12V_PROTECTED
- J1 pad A32: (no net) -> 12V_PROTECTED
- J1 pad A33: (no net) -> /V100_PCIE/V100_GND
- J1 pad A34: (no net) -> 12V_PROTECTED
- J1 pad A35: (no net) -> 12V_PROTECTED
- J1 pad A36: (no net) -> /V100_PCIE/V100_GND
- J1 pad A37: (no net) -> 12V_PROTECTED
- J1 pad A38: (no net) -> 12V_PROTECTED
- J1 pad A39: (no net) -> /V100_PCIE/V100_GND
- J1 pad A40: (no net) -> 12V_PROTECTED
- J1 pad B21: (no net) -> /V100_PCIE/V100_GND
- J1 pad B22: (no net) -> 12V_PROTECTED
- J1 pad B23: (no net) -> 12V_PROTECTED
- J1 pad B24: (no net) -> /V100_PCIE/V100_GND
- J1 pad B25: (no net) -> 12V_PROTECTED
- J1 pad B26: (no net) -> 12V_PROTECTED
- J1 pad B27: (no net) -> /V100_PCIE/V100_GND
- J1 pad B28: (no net) -> 12V_PROTECTED
- J1 pad B29: (no net) -> 12V_PROTECTED
- J1 pad B30: (no net) -> /V100_PCIE/V100_GND
- J1 pad B31: (no net) -> 12V_PROTECTED
- J1 pad B32: (no net) -> 12V_PROTECTED
- J1 pad B33: (no net) -> /V100_PCIE/V100_GND
- J1 pad B34: (no net) -> 12V_PROTECTED
- J1 pad B35: (no net) -> 12V_PROTECTED
- J1 pad B36: (no net) -> /V100_PCIE/V100_GND
- J1 pad B37: (no net) -> 12V_PROTECTED
- J1 pad B38: (no net) -> 12V_PROTECTED
- J1 pad B39: (no net) -> /V100_PCIE/V100_GND
- J1 pad B40: (no net) -> 12V_PROTECTED
- J1 pad C21: (no net) -> /V100_PCIE/V100_GND
- J1 pad C22: (no net) -> 12V_PROTECTED
- J1 pad C23: (no net) -> 12V_PROTECTED
- J1 pad C24: (no net) -> /V100_PCIE/V100_GND
- J1 pad C25: (no net) -> 12V_PROTECTED
- J1 pad C26: (no net) -> 12V_PROTECTED
- J1 pad C27: (no net) -> /V100_PCIE/V100_GND
- J1 pad C28: (no net) -> 12V_PROTECTED
- J1 pad C29: (no net) -> 12V_PROTECTED
- J1 pad C30: (no net) -> /V100_PCIE/V100_GND
- J1 pad C31: (no net) -> 12V_PROTECTED
- J1 pad C32: (no net) -> 12V_PROTECTED
- J1 pad C33: (no net) -> /V100_PCIE/V100_GND
- J1 pad C34: (no net) -> 12V_PROTECTED
- J1 pad C35: (no net) -> 12V_PROTECTED
- J1 pad C36: (no net) -> /V100_PCIE/V100_GND
- J1 pad C37: (no net) -> 12V_PROTECTED
- J1 pad C38: (no net) -> 12V_PROTECTED
- J1 pad C39: (no net) -> /V100_PCIE/V100_GND
- J1 pad C40: (no net) -> 12V_PROTECTED
- J1 pad D21: (no net) -> /V100_PCIE/V100_GND
- J1 pad D22: (no net) -> 12V_PROTECTED
- J1 pad D23: (no net) -> 12V_PROTECTED
- J1 pad D24: (no net) -> /V100_PCIE/V100_GND
- J1 pad D25: (no net) -> 12V_PROTECTED
- J1 pad D26: (no net) -> 12V_PROTECTED
- J1 pad D27: (no net) -> /V100_PCIE/V100_GND
- J1 pad D28: (no net) -> 12V_PROTECTED
- J1 pad D29: (no net) -> 12V_PROTECTED
- J1 pad D30: (no net) -> /V100_PCIE/V100_GND
- J1 pad D31: (no net) -> 12V_PROTECTED
- J1 pad D32: (no net) -> 12V_PROTECTED
- J1 pad D33: (no net) -> /V100_PCIE/V100_GND
- J1 pad D34: (no net) -> 12V_PROTECTED
- J1 pad D35: (no net) -> 12V_PROTECTED
- J1 pad D36: (no net) -> /V100_PCIE/V100_GND
- J1 pad D37: (no net) -> 12V_PROTECTED
- J1 pad D38: (no net) -> 12V_PROTECTED
- J1 pad D39: (no net) -> /V100_PCIE/V100_GND
- J1 pad D40: (no net) -> 12V_PROTECTED
- J1 pad E18: /STORAGE/BRIDGE_SATA_RX_N -> /V100_PCIE/V100_PERST
- J1 pad E21: (no net) -> /V100_PCIE/V100_GND
- J1 pad E22: (no net) -> 12V_PROTECTED
- J1 pad E23: (no net) -> 12V_PROTECTED
- J1 pad E24: (no net) -> /V100_PCIE/V100_GND
- J1 pad E25: (no net) -> 12V_PROTECTED
- J1 pad E26: (no net) -> 12V_PROTECTED
- J1 pad E27: (no net) -> /V100_PCIE/V100_GND
- J1 pad E28: (no net) -> 12V_PROTECTED
- J1 pad E29: (no net) -> 12V_PROTECTED
- J1 pad E30: (no net) -> /V100_PCIE/V100_GND
- J1 pad E31: (no net) -> 12V_PROTECTED
- J1 pad E32: (no net) -> 12V_PROTECTED
- J1 pad E33: (no net) -> /V100_PCIE/V100_GND
- J1 pad E34: (no net) -> 12V_PROTECTED
- J1 pad E35: (no net) -> 12V_PROTECTED
- J1 pad E36: (no net) -> /V100_PCIE/V100_GND
- J1 pad E37: (no net) -> 12V_PROTECTED
- J1 pad E38: (no net) -> 12V_PROTECTED
- J1 pad E39: (no net) -> /V100_PCIE/V100_GND
- J1 pad E40: (no net) -> 12V_PROTECTED
- J1 pad E7: /V100_PCIE/V100_PET0_N -> /V100_PCIE/V100_REFCLK_P
- J1 pad F21: (no net) -> /V100_PCIE/V100_GND
- J1 pad F22: (no net) -> 12V_PROTECTED
- J1 pad F23: (no net) -> 12V_PROTECTED
- J1 pad F24: (no net) -> /V100_PCIE/V100_GND
- J1 pad F25: (no net) -> 12V_PROTECTED
- J1 pad F26: (no net) -> 12V_PROTECTED
- J1 pad F27: (no net) -> /V100_PCIE/V100_GND
- J1 pad F28: (no net) -> 12V_PROTECTED
- J1 pad F29: (no net) -> 12V_PROTECTED
- J1 pad F30: (no net) -> /V100_PCIE/V100_GND
- J1 pad F31: (no net) -> 12V_PROTECTED
- J1 pad F32: (no net) -> 12V_PROTECTED
- J1 pad F33: (no net) -> /V100_PCIE/V100_GND
- J1 pad F34: (no net) -> 12V_PROTECTED
- J1 pad F35: (no net) -> 12V_PROTECTED
- J1 pad F36: (no net) -> /V100_PCIE/V100_GND
- J1 pad F37: (no net) -> 12V_PROTECTED
- J1 pad F38: (no net) -> 12V_PROTECTED
- J1 pad F39: (no net) -> /V100_PCIE/V100_GND
- J1 pad F40: (no net) -> 12V_PROTECTED
- J1 pad F7: /V100_PCIE/V100_PET0_P -> /V100_PCIE/V100_REFCLK_N
- J1 pad G1: /V100_PCIE/V100_REFCLK_N -> /V100_PCIE/V100_PET0_P
- J1 pad G2: /V100_PCIE/V100_REFCLK_P -> /V100_PCIE/V100_PET0_N
- J1 pad G21: (no net) -> /V100_PCIE/V100_GND
- J1 pad G22: (no net) -> 12V_PROTECTED
- J1 pad G23: (no net) -> 12V_PROTECTED
- J1 pad G24: (no net) -> /V100_PCIE/V100_GND
- J1 pad G25: (no net) -> 12V_PROTECTED
- J1 pad G26: (no net) -> 12V_PROTECTED
- J1 pad G27: (no net) -> /V100_PCIE/V100_GND
- J1 pad G28: (no net) -> 12V_PROTECTED
- J1 pad G29: (no net) -> 12V_PROTECTED
- J1 pad G30: (no net) -> /V100_PCIE/V100_GND
- J1 pad G31: (no net) -> 12V_PROTECTED
- J1 pad G32: (no net) -> 12V_PROTECTED
- J1 pad G33: (no net) -> /V100_PCIE/V100_GND
- J1 pad G34: (no net) -> 12V_PROTECTED
- J1 pad G35: (no net) -> 12V_PROTECTED
- J1 pad G36: (no net) -> /V100_PCIE/V100_GND
- J1 pad G37: (no net) -> 12V_PROTECTED
- J1 pad G38: (no net) -> 12V_PROTECTED
- J1 pad G39: (no net) -> /V100_PCIE/V100_GND
- J1 pad G40: (no net) -> 12V_PROTECTED
- J1 pad H21: (no net) -> /V100_PCIE/V100_GND
- J1 pad H22: (no net) -> 12V_PROTECTED
- J1 pad H23: (no net) -> 12V_PROTECTED
- J1 pad H24: (no net) -> /V100_PCIE/V100_GND
- J1 pad H25: (no net) -> 12V_PROTECTED
- J1 pad H26: (no net) -> 12V_PROTECTED
- J1 pad H27: (no net) -> /V100_PCIE/V100_GND
- J1 pad H28: (no net) -> 12V_PROTECTED
- J1 pad H29: (no net) -> 12V_PROTECTED
- J1 pad H30: (no net) -> /V100_PCIE/V100_GND
- J1 pad H31: (no net) -> 12V_PROTECTED
- J1 pad H32: (no net) -> 12V_PROTECTED
- J1 pad H33: (no net) -> /V100_PCIE/V100_GND
- J1 pad H34: (no net) -> 12V_PROTECTED
- J1 pad H35: (no net) -> 12V_PROTECTED
- J1 pad H36: (no net) -> /V100_PCIE/V100_GND
- J1 pad H37: (no net) -> 12V_PROTECTED
- J1 pad H38: (no net) -> 12V_PROTECTED
- J1 pad H39: (no net) -> /V100_PCIE/V100_GND
- J1 pad H40: (no net) -> 12V_PROTECTED
- J1 pad J21: (no net) -> /V100_PCIE/V100_GND
- J1 pad J22: (no net) -> 12V_PROTECTED
- J1 pad J23: (no net) -> 12V_PROTECTED
- J1 pad J24: (no net) -> /V100_PCIE/V100_GND
- J1 pad J25: (no net) -> 12V_PROTECTED
- J1 pad J26: (no net) -> 12V_PROTECTED
- J1 pad J27: (no net) -> /V100_PCIE/V100_GND
- J1 pad J28: (no net) -> 12V_PROTECTED
- J1 pad J29: (no net) -> 12V_PROTECTED
- J1 pad J30: (no net) -> /V100_PCIE/V100_GND
- J1 pad J31: (no net) -> 12V_PROTECTED
- J1 pad J32: (no net) -> 12V_PROTECTED
- J1 pad J33: (no net) -> /V100_PCIE/V100_GND
- J1 pad J34: (no net) -> 12V_PROTECTED
- J1 pad J35: (no net) -> 12V_PROTECTED
- J1 pad J36: (no net) -> /V100_PCIE/V100_GND
- J1 pad J37: (no net) -> 12V_PROTECTED
- J1 pad J38: (no net) -> 12V_PROTECTED
- J1 pad J39: (no net) -> /V100_PCIE/V100_GND
- J1 pad J40: (no net) -> 12V_PROTECTED
- J1 pad K21: (no net) -> /V100_PCIE/V100_GND
- J1 pad K22: (no net) -> 12V_PROTECTED
- J1 pad K23: (no net) -> 12V_PROTECTED
- J1 pad K24: (no net) -> /V100_PCIE/V100_GND
- J1 pad K25: (no net) -> 12V_PROTECTED
- J1 pad K26: (no net) -> 12V_PROTECTED
- J1 pad K27: (no net) -> /V100_PCIE/V100_GND
- J1 pad K28: (no net) -> 12V_PROTECTED
- J1 pad K29: (no net) -> 12V_PROTECTED
- J1 pad K30: (no net) -> /V100_PCIE/V100_GND
- J1 pad K31: (no net) -> 12V_PROTECTED
- J1 pad K32: (no net) -> 12V_PROTECTED
- J1 pad K33: (no net) -> /V100_PCIE/V100_GND
- J1 pad K34: (no net) -> 12V_PROTECTED
- J1 pad K35: (no net) -> 12V_PROTECTED
- J1 pad K36: (no net) -> /V100_PCIE/V100_GND
- J1 pad K37: (no net) -> 12V_PROTECTED
- J1 pad K38: (no net) -> 12V_PROTECTED
- J1 pad K39: (no net) -> /V100_PCIE/V100_GND
- J1 pad K40: (no net) -> 12V_PROTECTED

Commit message: start phase14 V100 power routing candidate
Connections:
- D1 pad 2: /POWER_INPUT/POWER_GND -> POWER_GND
- D2 pad 2: /POWER_INPUT/POWER_GND -> POWER_GND
- J1 pad A21: /V100_PCIE/V100_GND -> POWER_GND
- J1 pad A24: /V100_PCIE/V100_GND -> POWER_GND
- J1 pad A27: /V100_PCIE/V100_GND -> POWER_GND
- J1 pad A30: /V100_PCIE/V100_GND -> POWER_GND
- J1 pad A33: /V100_PCIE/V100_GND -> POWER_GND
- J1 pad A36: /V100_PCIE/V100_GND -> POWER_GND
- J1 pad A39: /V100_PCIE/V100_GND -> POWER_GND
- J1 pad B21: /V100_PCIE/V100_GND -> POWER_GND
- J1 pad B24: /V100_PCIE/V100_GND -> POWER_GND
- J1 pad B27: /V100_PCIE/V100_GND -> POWER_GND
- J1 pad B30: /V100_PCIE/V100_GND -> POWER_GND
- J1 pad B33: /V100_PCIE/V100_GND -> POWER_GND
- J1 pad B36: /V100_PCIE/V100_GND -> POWER_GND
- J1 pad B39: /V100_PCIE/V100_GND -> POWER_GND
- J1 pad C21: /V100_PCIE/V100_GND -> POWER_GND
- J1 pad C24: /V100_PCIE/V100_GND -> POWER_GND
- J1 pad C27: /V100_PCIE/V100_GND -> POWER_GND
- J1 pad C30: /V100_PCIE/V100_GND -> POWER_GND
- J1 pad C33: /V100_PCIE/V100_GND -> POWER_GND
- J1 pad C36: /V100_PCIE/V100_GND -> POWER_GND
- J1 pad C39: /V100_PCIE/V100_GND -> POWER_GND
- J1 pad D21: /V100_PCIE/V100_GND -> POWER_GND
- J1 pad D24: /V100_PCIE/V100_GND -> POWER_GND
- J1 pad D27: /V100_PCIE/V100_GND -> POWER_GND
- J1 pad D30: /V100_PCIE/V100_GND -> POWER_GND
- J1 pad D33: /V100_PCIE/V100_GND -> POWER_GND
- J1 pad D36: /V100_PCIE/V100_GND -> POWER_GND
- J1 pad D39: /V100_PCIE/V100_GND -> POWER_GND
- J1 pad E21: /V100_PCIE/V100_GND -> POWER_GND
- J1 pad E24: /V100_PCIE/V100_GND -> POWER_GND
- J1 pad E27: /V100_PCIE/V100_GND -> POWER_GND
- J1 pad E30: /V100_PCIE/V100_GND -> POWER_GND
- J1 pad E33: /V100_PCIE/V100_GND -> POWER_GND
- J1 pad E36: /V100_PCIE/V100_GND -> POWER_GND
- J1 pad E39: /V100_PCIE/V100_GND -> POWER_GND
- J1 pad F21: /V100_PCIE/V100_GND -> POWER_GND
- J1 pad F24: /V100_PCIE/V100_GND -> POWER_GND
- J1 pad F27: /V100_PCIE/V100_GND -> POWER_GND
- J1 pad F30: /V100_PCIE/V100_GND -> POWER_GND
- J1 pad F33: /V100_PCIE/V100_GND -> POWER_GND
- J1 pad F36: /V100_PCIE/V100_GND -> POWER_GND
- J1 pad F39: /V100_PCIE/V100_GND -> POWER_GND
- J1 pad G21: /V100_PCIE/V100_GND -> POWER_GND
- J1 pad G24: /V100_PCIE/V100_GND -> POWER_GND
- J1 pad G27: /V100_PCIE/V100_GND -> POWER_GND
- J1 pad G30: /V100_PCIE/V100_GND -> POWER_GND
- J1 pad G33: /V100_PCIE/V100_GND -> POWER_GND
- J1 pad G36: /V100_PCIE/V100_GND -> POWER_GND
- J1 pad G39: /V100_PCIE/V100_GND -> POWER_GND
- J1 pad H21: /V100_PCIE/V100_GND -> POWER_GND
- J1 pad H24: /V100_PCIE/V100_GND -> POWER_GND
- J1 pad H27: /V100_PCIE/V100_GND -> POWER_GND
- J1 pad H30: /V100_PCIE/V100_GND -> POWER_GND
- J1 pad H33: /V100_PCIE/V100_GND -> POWER_GND
- J1 pad H36: /V100_PCIE/V100_GND -> POWER_GND
- J1 pad H39: /V100_PCIE/V100_GND -> POWER_GND
- J1 pad J21: /V100_PCIE/V100_GND -> POWER_GND
- J1 pad J24: /V100_PCIE/V100_GND -> POWER_GND
- J1 pad J27: /V100_PCIE/V100_GND -> POWER_GND
- J1 pad J30: /V100_PCIE/V100_GND -> POWER_GND
- J1 pad J33: /V100_PCIE/V100_GND -> POWER_GND
- J1 pad J36: /V100_PCIE/V100_GND -> POWER_GND
- J1 pad J39: /V100_PCIE/V100_GND -> POWER_GND
- J1 pad K21: /V100_PCIE/V100_GND -> POWER_GND
- J1 pad K24: /V100_PCIE/V100_GND -> POWER_GND
- J1 pad K27: /V100_PCIE/V100_GND -> POWER_GND
- J1 pad K30: /V100_PCIE/V100_GND -> POWER_GND
- J1 pad K33: /V100_PCIE/V100_GND -> POWER_GND
- J1 pad K36: /V100_PCIE/V100_GND -> POWER_GND
- J1 pad K39: /V100_PCIE/V100_GND -> POWER_GND
- J5 pad 2: /POWER_INPUT/POWER_GND -> POWER_GND
- J6 pad 2: /POWER_INPUT/POWER_GND -> POWER_GND
- U1 pad 2: /POWER_INPUT/POWER_GND -> POWER_GND
- U2 pad 2: /POWER_INPUT/POWER_GND -> POWER_GND
