File: pisxme/reva-clean/ACREAGE_ETHERNET_PHASE17.kicad_pcb (KiCad board)
At the start: 6 copper layers, 300 x 180 mm, 72 parts, among them J1 74221-101LF, J2 A70-112-331N126, J3 JAE SM3ZS067U410ABR1000 B-key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, J4 Amphenol 10171746-00021LF USB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, J5 0039300020, J6 0039300020, J7 Raspberry-Pi-5-Compute-Module, Q1 CSD19536KCS, Q2 CSD19536KCS, U1 LM74700QDBVRQ1, U2 LM74700QDBVRQ1, U3 TPSM63606RDLR, U4 TPSM63606RDLR, U5 TPSM63606RDLR, U6 TPD4E004DRYR, U7 TUSB9261IPVP, U8 Texas_DRT_3, U9 TPD4E004DRYR

Commit message: docs: publish Phase 17 blocker evidence
Parts:
- moved J2 268.7 mm to (12.0, 120.0)
- moved U6 231.4 mm to (25.0, 99.0), turned to 180 degrees
- moved U9 230.1 mm to (25.0, 106.0), turned to 180 degrees
Routing:
- net CM5_GBE_TD1_P: track 0.00 -> 16.3 mm, vias 0 -> 1
- net CM5_GBE_TD0_N: track 0.00 -> 16.3 mm, vias 0 -> 1
- net CM5_GBE_TD2_N: track 0.00 -> 10.8 mm
- net CM5_GBE_TD3_P: track 0.00 -> 10.7 mm
- net CM5_GBE_TD1_N: track 0.00 -> 10.4 mm, vias 0 -> 1
- net CM5_GBE_TD0_P: track 0.00 -> 10.4 mm, vias 0 -> 1
- net CM5_GBE_TD2_P: track 0.00 -> 9.41 mm
- net CM5_GBE_TD3_N: track 0.00 -> 9.22 mm
Changed lines of the file:
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@@
 	(footprint "TPD4E004DRYR_WSON6"
 		(layer "F.Cu")
-		(at 250 58)
+		(at 25 106 180)
 		(descr "TPD4E004DRYR; package outline is datasheet-derived and requires final fab-library review")
 		(property "Reference" "U9"
-			(at 0 -1.75 0)
+			(at 0 -1.75 180)
 			(layer "F.SilkS")
 			(effects
@@
 		)
 		(property "Value" "TPD4E004DRYR"
-			(at 0 1.75 0)
+			(at 0 1.75 180)
 			(layer "F.Fab")
 			(hide yes)
@@
 		)
 		(property "Datasheet" ""
-			(at 0 0 0)
+			(at 0 0 180)
 			(layer "F.Fab")
 			(hide yes)
@@
 		)
 		(property "Description" ""
-			(at 0 0 0)
+			(at 0 0 180)
 			(layer "F.Fab")
 			(hide yes)
@@
 		)
 		(pad "1" smd roundrect
-			(at -0.75 -0.75)
+			(at -0.75 -0.75 180)
 			(size 0.28 0.28)
 			(layers "F.Cu" "F.Mask" "F.Paste")
@@
 		)
 		(pad "2" smd roundrect
-			(at 0.75 -0.75 90)
+			(at 0.75 -0.75 270)
 			(size 0.28 0.28)
 			(layers "F.Cu" "F.Mask" "F.Paste")
@@
 		)
 		(pad "3" smd roundrect
-			(at 0.75 0.75 180)
+			(at 0.75 0.75)
 			(size 0.28 0.28)
 			(layers "F.Cu" "F.Mask" "F.Paste")
@@
 		)
 		(pad "4" smd roundrect
-			(at -0.75 0.75 270)
+			(at -0.75 0.75 90)
 			(size 0.28 0.28)
 			(layers "F.Cu" "F.Mask" "F.Paste")
@@
 		)
 		(pad "5" smd roundrect
-			(at -0.25 0.75 270)
+			(at -0.25 0.75 90)
 			(size 0.28 0.28)
 			(layers "F.Cu" "F.Mask" "F.Paste")
@@
 		)
 		(pad "6" smd roundrect
-			(at 0.25 0.75 270)
+			(at 0.25 0.75 90)
 			(size 0.28 0.28)
 			(layers "F.Cu" "F.Mask" "F.Paste")
@@
 	(footprint "TPD4E004DRYR_WSON6"
 		(layer "F.Cu")
-		(at 250 45)
+		(at 25 99 180)
 		(descr "TPD4E004DRYR; package outline is datasheet-derived and requires final fab-library review")
 		(property "Reference" "U6"
-			(at 0 -1.75 0)
+			(at 0 -1.75 180)
 			(layer "F.SilkS")
 			(effects
@@
 		)
 		(property "Value" "TPD4E004DRYR"
-			(at 0 1.75 0)
+			(at 0 1.75 180)
 			(layer "F.Fab")
 			(hide yes)
@@
 		)
 		(property "Datasheet" ""
-			(at 0 0 0)
+			(at 0 0 180)
 			(layer "F.Fab")
 			(hide yes)
@@
 		)
 		(property "Description" ""
-			(at 0 0 0)
+			(at 0 0 180)
 			(layer "F.Fab")
 			(hide yes)
@@
 		)
 		(pad "1" smd roundrect
-			(at -0.75 -0.75)
+			(at -0.75 -0.75 180)
 			(size 0.28 0.28)
 			(layers "F.Cu" "F.Mask" "F.Paste")
@@
 		)
 		(pad "2" smd roundrect
-			(at 0.75 -0.75 90)
+			(at 0.75 -0.75 270)
 			(size 0.28 0.28)
 			(layers "F.Cu" "F.Mask" "F.Paste")
@@
 		)
 		(pad "3" smd roundrect
-			(at 0.75 0.75 180)
+			(at 0.75 0.75)
 			(size 0.28 0.28)
 			(layers "F.Cu" "F.Mask" "F.Paste")
@@
 		)
 		(pad "4" smd roundrect
-			(at -0.75 0.75 270)
+			(at -0.75 0.75 90)
 			(size 0.28 0.28)
 			(layers "F.Cu" "F.Mask" "F.Paste")
@@
 		)
 		(pad "5" smd roundrect
-			(at -0.25 0.75 270)
+			(at -0.25 0.75 90)
 			(size 0.28 0.28)
 			(layers "F.Cu" "F.Mask" "F.Paste")
@@
 		)
 		(pad "6" smd roundrect
-			(at 0.25 0.75 270)
+			(at 0.25 0.75 90)
 			(size 0.28 0.28)
 			(layers "F.Cu" "F.Mask" "F.Paste")
@@
 	(footprint "EDAC_A70_112_331N126"
 		(layer "F.Cu")
-		(at 270 45)
+		(at 12 120)
 		(descr "EDAC A70-112-331N126; EDAC drawing via Mouser; no 3D model attached")
 		(tags "RJ45 MagJack Ethernet PoE EDAC A70-112-331N126")
@@
 	)
 	(segment
+		(start 32.96 100.7)
+		(end 25.75 106.75)
+		(width 0.13208)
+		(layer "F.Cu")
+		(net "CM5_GBE_TD2_P")
+	)
+	(segment
+		(start 32.96 100.3)
+		(end 24.25 106.75)
+		(width 0.13208)
+		(layer "F.Cu")
+		(net "CM5_GBE_TD2_N")
+	)
+	(segment
+		(start 32.96 99.1)
+		(end 24.25 105.25)
+		(width 0.13208)
+		(layer "F.Cu")
+		(net "CM5_GBE_TD3_P")
+	)
+	(segment
+		(start 32.96 99.5)
+		(end 25.75 105.25)
+		(width 0.13208)
+		(layer "F.Cu")
+		(net "CM5_GBE_TD3_N")
+	)
+	(segment
+		(start 29 99.75)
+		(end 25.75 99.75)
+		(width 0.13208)
+		(layer "F.Cu")
+		(net "CM5_GBE_TD0_P")
+	)
+	(via
+		(at 29 99.75)
+		(size 0.5)
+		(drill 0.3)
+		(layers "F.Cu" "B.Cu")
+		(net "CM5_GBE_TD0_P")
+	)
+	(segment
+		(start 36.04 100.7)
+		(end 29 99.75)
+		(width 0.13208)
+		(layer "B.Cu")
+		(net "CM5_GBE_TD0_P")
+	)
+	(segment
+		(start 22 99.75)
+		(end 24.25 99.75)
+		(width 0.13208)
+		(layer "F.Cu")
+		(net "CM5_GBE_TD0_N")
+	)
+	(via
+		(at 22 99.75)
+		(size 0.5)
+		(drill 0.3)
+		(layers "F.Cu" "B.Cu")
+		(net "CM5_GBE_TD0_N")
+	)
+	(segment
+		(start 36.04 100.3)
+		(end 22 99.75)
+		(width 0.13208)
+		(layer "B.Cu")
+		(net "CM5_GBE_TD0_N")
+	)
+	(segment
+		(start 22 98.25)
+		(end 24.25 98.25)
+		(width 0.13208)
+		(layer "F.Cu")
+		(net "CM5_GBE_TD1_P")
+	)
+	(via
+		(at 22 98.25)
+		(size 0.5)
+		(drill 0.3)
+		(layers "F.Cu" "B.Cu")
+		(net "CM5_GBE_TD1_P")
+	)
+	(segment
+		(start 36.04 99.1)
+		(end 22 98.25)
+		(width 0.13208)
+		(layer "B.Cu")
+		(net "CM5_GBE_TD1_P")
+	)
+	(segment
+		(start 29 98.25)
+		(end 25.75 98.25)
+		(width 0.13208)
+		(layer "F.Cu")
+		(net "CM5_GBE_TD1_N")
+	)
+	(via
+		(at 29 98.25)
+		(size 0.5)
+		(drill 0.3)
+		(layers "F.Cu" "B.Cu")
+		(net "CM5_GBE_TD1_N")
+	)
+	(segment
+		(start 36.04 99.5)
+		(end 29 98.25)
+		(width 0.13208)
+		(layer "B.Cu")
+		(net "CM5_GBE_TD1_N")
+	)
+	(segment
