File: pisxme/reva-clean/ACREAGE_U3_CONTROLS_PHASE15.kicad_pcb (KiCad board)
At the start: 6 copper layers, 300 x 180 mm, 72 parts, among them J1 74221-101LF, J2 A70-112-331N126, J3 JAE SM3ZS067U410ABR1000 B-key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, J4 Amphenol 10171746-00021LF USB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, J5 0039300020, J6 0039300020, J7 Raspberry-Pi-5-Compute-Module, Q1 CSD19536KCS, Q2 CSD19536KCS, U1 LM74700QDBVRQ1, U2 LM74700QDBVRQ1, U3 TPSM63606RDLR, U4 TPSM63606RDLR, U5 TPSM63606RDLR, U6 TPD4E004DRYR, U7 TUSB9261IPVP, U8 Texas_DRT_3, U9 TPD4E004DRYR

Commit message: phase15: tie regulator output lands
Routing:
- net /REGULATORS/CM5_5V: track 131.6 -> 152.7 mm

Commit message: phase16: close PCIe net authority
Connections:
- J1 pad A2: /V100_PCIE/V100_PER0_P -> /CORE_CM5/CM5_PER0_P
- J1 pad A3: /V100_PCIE/V100_PER0_N -> /CORE_CM5/CM5_PER0_N
- J1 pad E18: /V100_PCIE/V100_PERST -> /CORE_CM5/CM5_PERST
- J1 pad E7: /V100_PCIE/V100_REFCLK_P -> /CORE_CM5/CM5_REFCLK_P
- J1 pad F7: /V100_PCIE/V100_REFCLK_N -> /CORE_CM5/CM5_REFCLK_N

Commit message: phase16: close PET0 source-side authority
Connections:
- C1 pad 1: /V100_PCIE/CM5_PET0_P -> /CORE_CM5/CM5_PET0_P
- C2 pad 1: /V100_PCIE/CM5_PET0_N -> /CORE_CM5/CM5_PET0_N

Commit message: docs: publish Phase 17 blocker evidence
Connections:
- J2 pad 11: /ETHERNET/CM5_GBE_TD3_N -> CM5_GBE_TD3_N
- J2 pad 12: /ETHERNET/CM5_GBE_TD3_P -> CM5_GBE_TD3_P
- J2 pad 13: /ETHERNET/CM5_GBE_TD2_N -> CM5_GBE_TD2_N
- J2 pad 14: /ETHERNET/CM5_GBE_TD2_P -> CM5_GBE_TD2_P
- J2 pad 15: /ETHERNET/CM5_GBE_TD1_N -> CM5_GBE_TD1_N
- J2 pad 16: /ETHERNET/CM5_GBE_TD1_P -> CM5_GBE_TD1_P
- J2 pad 17: /ETHERNET/CM5_GBE_TD0_N -> CM5_GBE_TD0_N
- J2 pad 18: /ETHERNET/CM5_GBE_TD0_P -> CM5_GBE_TD0_P
- J7 pad 10: /CORE_CM5/CM5_GBE_TD0_N -> CM5_GBE_TD0_N
- J7 pad 11: /CORE_CM5/CM5_GBE_TD2_P -> CM5_GBE_TD2_P
- J7 pad 12: /CORE_CM5/CM5_GBE_TD0_P -> CM5_GBE_TD0_P
- J7 pad 3: /CORE_CM5/CM5_GBE_TD3_P -> CM5_GBE_TD3_P
- J7 pad 4: /CORE_CM5/CM5_GBE_TD1_P -> CM5_GBE_TD1_P
- J7 pad 5: /CORE_CM5/CM5_GBE_TD3_N -> CM5_GBE_TD3_N
- J7 pad 6: /CORE_CM5/CM5_GBE_TD1_N -> CM5_GBE_TD1_N
- J7 pad 9: /CORE_CM5/CM5_GBE_TD2_N -> CM5_GBE_TD2_N
- U6 pad 1: /ETHERNET/ETH_GND -> CM5_GBE_TD0_P
- U6 pad 2: /ETHERNET/ETH_POWER -> CM5_GBE_TD0_N
- U6 pad 3: /ETHERNET/CM5_GBE_TD1_N -> CM5_GBE_TD1_P
- U6 pad 4: /ETHERNET/CM5_GBE_TD1_P -> CM5_GBE_TD1_N
- U6 pad 5: /ETHERNET/CM5_GBE_TD0_N -> /ETHERNET/ETH_POWER
- U6 pad 6: /ETHERNET/CM5_GBE_TD0_P -> /ETHERNET/ETH_GND
- U9 pad 1: /ETHERNET/ETH_GND -> CM5_GBE_TD2_P
- U9 pad 2: /ETHERNET/ETH_POWER -> CM5_GBE_TD2_N
- U9 pad 3: /ETHERNET/CM5_GBE_TD3_N -> CM5_GBE_TD3_P
- U9 pad 4: /ETHERNET/CM5_GBE_TD3_P -> CM5_GBE_TD3_N
- U9 pad 5: /ETHERNET/CM5_GBE_TD2_N -> /ETHERNET/ETH_POWER
- U9 pad 6: /ETHERNET/CM5_GBE_TD2_P -> /ETHERNET/ETH_GND
