File: pisxme/reva-clean/ACREAGE_CM5IO_RIGHT_CHANNEL_PHASE17.kicad_pcb (KiCad board)
At the start: 6 copper layers, 300 x 180 mm, 72 parts, among them J1 74221-101LF, J2 A70-112-331N126, J3 JAE SM3ZS067U410ABR1000 B-key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, J4 Amphenol 10171746-00021LF USB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, J5 0039300020, J6 0039300020, J7 Raspberry-Pi-5-Compute-Module, Q1 CSD19536KCS, Q2 CSD19536KCS, U1 LM74700QDBVRQ1, U2 LM74700QDBVRQ1, U3 TPSM63606RDLR, U4 TPSM63606RDLR, U5 TPSM63606RDLR, U6 TPD4EUSB30, U7 TUSB9261IPVP, U8 Texas_DRT_3, U9 TPD4EUSB30

Commit message: phase17: correct ethernet mode coordinates
Parts:
- moved U6 241.3 mm to (273.6, 32.2)
- moved U9 241.3 mm to (267.6, 32.2)
- moved J2 241.3 mm to (270.0, 20.0)

Commit message: phase17: record right-channel bcu trial
Routing:
- net CM5_GBE_TD0_N: track 311.4 -> 276.2 mm, vias 0 -> 2
- net CM5_GBE_TD0_P: track 307.2 -> 272.1 mm, vias 0 -> 2
- net CM5_GBE_TD2_N: track 308.9 -> 274.3 mm, vias 0 -> 2
- net CM5_GBE_TD2_P: track 308.4 -> 273.9 mm, vias 0 -> 2
- net CM5_GBE_TD1_P: track 312.2 -> 278.6 mm, vias 0 -> 2
- net CM5_GBE_TD1_N: track 313.3 -> 279.6 mm, vias 0 -> 2
- net CM5_GBE_TD3_P: track 309.3 -> 276.4 mm, vias 0 -> 2
- net CM5_GBE_TD3_N: track 309.0 -> 276.0 mm, vias 0 -> 2
