File: pisxme/reva-clean/ACREAGE_PHASE17_WEST_PERIMETER_MDI.kicad_pcb (KiCad board)
At the start: 6 copper layers, 300 x 180 mm, 81 parts, among them J1 74221-101LF, J2 A70-112-331N126, J3 JAE SM3ZS067U410ABR1000 B-key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, J4 Amphenol 10171746-00021LF USB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, J5 0039300020, J6 0039300020, J7 Raspberry-Pi-5-Compute-Module, Q1 CSD19536KCS, Q2 CSD19536KCS, U1 LM74700QDBVRQ1, U2 LM74700QDBVRQ1, U3 TPSM63606RDLR, U4 TPSM63606RDLR, U5 TPSM63606RDLR, U6 TPD4EUSB30, U7 TUSB9261IPVP, U8 Texas_DRT_3, U9 TPD4EUSB30

Commit message: phase17: record package-aware dogbone retry
Routing:
- net CM5_GBE_TD1_P: track 404.8 -> 401.8 mm
- net CM5_GBE_TD0_N: track 424.4 -> 421.4 mm
- net CM5_GBE_TD0_P: track 431.9 -> 428.9 mm
- net CM5_GBE_TD1_N: track 407.9 -> 404.9 mm

Commit message: phase17: record source column layer split retry
Routing:
- net CM5_GBE_TD0_P: track 428.9 -> 377.6 mm, vias 0 -> 3
- net CM5_GBE_TD0_N: track 421.4 -> 374.1 mm, vias 0 -> 3
- net CM5_GBE_TD1_N: track 404.9 -> 361.6 mm, vias 0 -> 3
- net CM5_GBE_TD1_P: track 401.8 -> 362.5 mm, vias 0 -> 3
- net CM5_GBE_TD3_P: track 407.1 -> 403.1 mm
- net CM5_GBE_TD3_N: track 412.7 -> 408.7 mm
- net CM5_GBE_TD2_N: track 426.7 -> 422.7 mm
- net CM5_GBE_TD2_P: track 434.2 -> 430.2 mm
