File: pisxme/reva-clean/ACREAGE_PHASE17_COLOCATED_CT4_SPLIT.kicad_pcb (KiCad board)
At the start: 6 copper layers, 300 x 180 mm, 81 parts, among them J1 74221-101LF, J2 A70-112-331N126, J3 JAE SM3ZS067U410ABR1000 B-key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, J4 Amphenol 10171746-00021LF USB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, J5 0039300020, J6 0039300020, J7 Raspberry-Pi-5-Compute-Module, Q1 CSD19536KCS, Q2 CSD19536KCS, U1 LM74700QDBVRQ1, U2 LM74700QDBVRQ1, U3 TPSM63606RDLR, U4 TPSM63606RDLR, U5 TPSM63606RDLR, U6 TPD4EUSB30, U7 TUSB9261IPVP, U8 Texas_DRT_3, U9 TPD4EUSB30

Commit message: phase17: close ethernet routing gate
Parts:
- removed MECH_V100: REV_A_EMPIRICAL_RISK: 150x95mm cooler/backplate envelope, V100_COOLER_BACKPLATE_ENVELOPE
Routing:
- net /ETHERNET/ETH_CT4: vias 2 -> 1
