File: pisxme/reva-clean/PHASE24_CLOCK_SWEEP_nearwest.kicad_pcb (KiCad board)
At the start: 6 copper layers, 300 x 180 mm, 94 parts, among them J1 74221-101LF, J2 A70-112-331N126, J3 JAE SM3ZS067U410ABR1000 B-key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, J4 Amphenol 10171746-00021LF USB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, J5 0039300020, J6 0039300020, J7 Raspberry-Pi-5-Compute-Module, Q1 CSD19536KCS, Q2 CSD19536KCS, U1 LM74700QDBVRQ1, U2 LM74700QDBVRQ1, U3 TPSM63606RDLR, U4 TPSM63606RDLR, U5 TPSM63606RDLR, U6 TPD4EUSB30, U7 TUSB9261IPVP, U8 Texas_DRT_3, U9 TPD4EUSB30

Commit message: phase24 reject clock rotation trial
Parts:
- turned Y1 to 90 degrees
Routing:
- net /STORAGE/BRIDGE_XO: track 20.6 -> 22.8 mm
- net /STORAGE/BRIDGE_XI: track 23.9 -> 25.6 mm
- net /STORAGE/BRIDGE_VSSOSC: track 21.9 -> 20.2 mm
Changed lines of the file:
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@@
 		(embedded_fonts no)
 	)
+	(footprint "Crystal_3225_4Pad"
+		(layer "F.Cu")
+		(at 108 130 90)
+		(descr "3.2 x 2.5 mm 4-pad crystal; verify vendor pad numbering before release")
+		(property "Reference" "Y1"
+			(at 0 0 90)
+			(layer "F.SilkS")
+			(effects
+				(font
+					(size 1.27 1.27)
+				)
+			)
+		)
+		(property "Value" ""
+			(at 0 0 90)
+			(layer "F.Fab")
+			(effects
+				(font
+					(size 1.27 1.27)
+				)
+			)
+		)
+		(property "Datasheet" ""
+			(at 0 0 90)
+			(layer "F.Fab")
+			(hide yes)
+			(effects
+				(font
+					(size 1.27 1.27)
+				)
+			)
+		)
+		(property "Description" ""
+			(at 0 0 90)
+			(layer "F.Fab")
+			(hide yes)
+			(effects
+				(font
+					(size 1.27 1.27)
+				)
+			)
+		)
+		(duplicate_pad_numbers_are_jumpers no)
+		(fp_rect
+			(start -1.6 -1.25)
+			(end 1.6 1.25)
+			(stroke
+				(width 0.12)
+				(type default)
+			)
+			(fill no)
+			(layer "F.SilkS")
+		)
+		(fp_rect
+			(start -1.7 -1.35)
+			(end 1.7 1.35)
+			(stroke
+				(width 0.05)
+				(type default)
+			)
+			(fill no)
+			(layer "F.CrtYd")
+		)
+		(pad "1" smd roundrect
+			(at -1.1 -0.85 90)
+			(size 1.2 0.9)
+			(layers "F.Cu" "F.Mask" "F.Paste")
+			(roundrect_rratio 0.2)
+			(net "/STORAGE/BRIDGE_XI")
+		)
+		(pad "2" smd roundrect
+			(at -1.1 0.85 90)
+			(size 1.2 0.9)
+			(layers "F.Cu" "F.Mask" "F.Paste")
+			(roundrect_rratio 0.2)
+			(net "/STORAGE/BRIDGE_VSSOSC")
+		)
+		(pad "3" smd roundrect
+			(at 1.1 0.85 90)
+			(size 1.2 0.9)
+			(layers "F.Cu" "F.Mask" "F.Paste")
+			(roundrect_rratio 0.2)
+			(net "/STORAGE/BRIDGE_XO")
+		)
+		(pad "4" smd roundrect
+			(at 1.1 -0.85 90)
+			(size 1.2 0.9)
+			(layers "F.Cu" "F.Mask" "F.Paste")
+			(roundrect_rratio 0.2)
+			(net "/STORAGE/BRIDGE_VSSOSC")
+		)
+		(embedded_fonts no)
+	)
 	(footprint "Texas_DRT_3"
 		(layer "F.Cu")
@@
 		(embedded_fonts no)
 	)
-	(footprint "Crystal_3225_4Pad"
-		(layer "F.Cu")
-		(at 108 130)
-		(descr "3.2 x 2.5 mm 4-pad crystal; verify vendor pad numbering before release")
-		(property "Reference" "Y1"
-			(at 0 0 0)
-			(layer "F.SilkS")
-			(effects
-				(font
-					(size 1.27 1.27)
-				)
-			)
-		)
-		(property "Value" ""
-			(at 0 0 0)
-			(layer "F.Fab")
-			(effects
-				(font
-					(size 1.27 1.27)
-				)
-			)
-		)
-		(property "Datasheet" ""
-			(at 0 0 0)
-			(layer "F.Fab")
-			(hide yes)
-			(effects
-				(font
-					(size 1.27 1.27)
-				)
-			)
-		)
-		(property "Description" ""
-			(at 0 0 0)
-			(layer "F.Fab")
-			(hide yes)
-			(effects
-				(font
-					(size 1.27 1.27)
-				)
-			)
-		)
-		(duplicate_pad_numbers_are_jumpers no)
-		(fp_rect
-			(start -1.6 -1.25)
-			(end 1.6 1.25)
-			(stroke
-				(width 0.12)
-				(type default)
-			)
-			(fill no)
-			(layer "F.SilkS")
-		)
-		(fp_rect
-			(start -1.7 -1.35)
-			(end 1.7 1.35)
-			(stroke
-				(width 0.05)
-				(type default)
-			)
-			(fill no)
-			(layer "F.CrtYd")
-		)
-		(pad "1" smd roundrect
-			(at -1.1 -0.85)
-			(size 1.2 0.9)
-			(layers "F.Cu" "F.Mask" "F.Paste")
-			(roundrect_rratio 0.2)
-			(net "/STORAGE/BRIDGE_XI")
-		)
-		(pad "2" smd roundrect
-			(at -1.1 0.85)
-			(size 1.2 0.9)
-			(layers "F.Cu" "F.Mask" "F.Paste")
-			(roundrect_rratio 0.2)
-			(net "/STORAGE/BRIDGE_VSSOSC")
-		)
-		(pad "3" smd roundrect
-			(at 1.1 0.85)
-			(size 1.2 0.9)
-			(layers "F.Cu" "F.Mask" "F.Paste")
-			(roundrect_rratio 0.2)
-			(net "/STORAGE/BRIDGE_XO")
-		)
-		(pad "4" smd roundrect
-			(at 1.1 -0.85)
-			(size 1.2 0.9)
-			(layers "F.Cu" "F.Mask" "F.Paste")
-			(roundrect_rratio 0.2)
-			(net "/STORAGE/BRIDGE_VSSOSC")
-		)
-		(embedded_fonts no)
-	)
 	(footprint "R_0402_1005Metric"
 		(layer "F.Cu")
@@
 	(segment
 		(start 124 129)
-		(end 106.9 129)
+		(end 107.15 129)
 		(width 0.1321)
 		(layer "B.Cu")
@@
 	)
 	(segment
-		(start 106.9 129)
-		(end 106.9 129.15)
+		(start 107.15 129)
+		(end 107.15 131.1)
 		(width 0.1321)
 		(layer "B.Cu")
@@
 	)
 	(segment
-		(start 122.5 135.5)
-		(end 122.5 133.5)
+		(start 122.5 133.5)
+		(end 122.5 130.5)
 		(width 0.1321)
 		(layer "F.Cu")
@@
 	)
 	(segment
-		(start 122.5 133.5)
-		(end 122.5 130.5)
+		(start 122.5 135.5)
+		(end 122.5 133.5)
 		(width 0.1321)
 		(layer "F.Cu")
@@
 	)
 	(segment
-		(start 122.5 130)
-		(end 106.9 130)
+		(start 108.85 130)
+		(end 108.85 131.1)
 		(width 0.1321)
 		(layer "B.Cu")
@@
 	)
 	(segment
-		(start 122.5 130.5)
-		(end 122.5 130)
+		(start 122.5 130)
+		(end 108.85 130)
 		(width 0.1321)
 		(layer "B.Cu")
@@
 	)
 	(segment
-		(start 106.9 130)
-		(end 106.9 130.85)
+		(start 122.5 130.5)
+		(end 122.5 130)
 		(width 0.1321)
 		(layer "B.Cu")
@@
 	)
 	(segment
-		(start 122 132.5)
-		(end 122 129.5)
+		(start 122 135.5)
+		(end 122 132.5)
 		(width 0.1321)
 		(layer "F.Cu")
@@
 	)
 	(segment
-		(start 122 135.5)
-		(end 122 132.5)
+		(start 122 132.5)
+		(end 122 129.5)
 		(width 0.1321)
 		(layer "F.Cu")
@@
 	)
 	(segment
-		(start 109.1 131)
-		(end 109.1 130.85)
+		(start 108.85 131)
+		(end 108.85 128.9)
 		(width 0.1321)
 		(layer "B.Cu")
@@
 	)
 	(segment
-		(start 122 131)
-		(end 109.1 131)
+		(start 122 129.5)
+		(end 122 131)
 		(width 0.1321)
 		(layer "B.Cu")
@@
 	)
 	(segment
-		(start 122 129.5)
-		(end 122 131)
+		(start 122 131)
+		(end 108.85 131)
 		(width 0.1321)
 		(layer "B.Cu")

Commit message: phase24 correct clock sweep evidence
Parts:
- turned Y1 to 0 degrees
Routing:
- net /STORAGE/BRIDGE_XI: track 25.6 -> 29.9 mm
- net /STORAGE/BRIDGE_XO: track 22.8 -> 21.6 mm
- net /STORAGE/BRIDGE_VSSOSC: track 20.2 -> 19.8 mm, vias 1 -> 0
Changed lines of the file:
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@@
 		(embedded_fonts no)
 	)
-	(footprint "Crystal_3225_4Pad"
-		(layer "F.Cu")
-		(at 108 130 90)
-		(descr "3.2 x 2.5 mm 4-pad crystal; verify vendor pad numbering before release")
-		(property "Reference" "Y1"
-			(at 0 0 90)
-			(layer "F.SilkS")
-			(effects
-				(font
-					(size 1.27 1.27)
-				)
-			)
-		)
-		(property "Value" ""
-			(at 0 0 90)
-			(layer "F.Fab")
-			(effects
-				(font
-					(size 1.27 1.27)
-				)
-			)
-		)
-		(property "Datasheet" ""
-			(at 0 0 90)
-			(layer "F.Fab")
-			(hide yes)
-			(effects
-				(font
-					(size 1.27 1.27)
-				)
-			)
-		)
-		(property "Description" ""
-			(at 0 0 90)
-			(layer "F.Fab")
-			(hide yes)
-			(effects
-				(font
-					(size 1.27 1.27)
-				)
-			)
-		)
-		(duplicate_pad_numbers_are_jumpers no)
-		(fp_rect
-			(start -1.6 -1.25)
-			(end 1.6 1.25)
-			(stroke
-				(width 0.12)
-				(type default)
-			)
-			(fill no)
-			(layer "F.SilkS")
-		)
-		(fp_rect
-			(start -1.7 -1.35)
-			(end 1.7 1.35)
-			(stroke
-				(width 0.05)
-				(type default)
-			)
-			(fill no)
-			(layer "F.CrtYd")
-		)
-		(pad "1" smd roundrect
-			(at -1.1 -0.85 90)
-			(size 1.2 0.9)
-			(layers "F.Cu" "F.Mask" "F.Paste")
-			(roundrect_rratio 0.2)
-			(net "/STORAGE/BRIDGE_XI")
-		)
-		(pad "2" smd roundrect
-			(at -1.1 0.85 90)
-			(size 1.2 0.9)
-			(layers "F.Cu" "F.Mask" "F.Paste")
-			(roundrect_rratio 0.2)
-			(net "/STORAGE/BRIDGE_VSSOSC")
-		)
-		(pad "3" smd roundrect
-			(at 1.1 0.85 90)
-			(size 1.2 0.9)
-			(layers "F.Cu" "F.Mask" "F.Paste")
-			(roundrect_rratio 0.2)
-			(net "/STORAGE/BRIDGE_XO")
-		)
-		(pad "4" smd roundrect
-			(at 1.1 -0.85 90)
-			(size 1.2 0.9)
-			(layers "F.Cu" "F.Mask" "F.Paste")
-			(roundrect_rratio 0.2)
-			(net "/STORAGE/BRIDGE_VSSOSC")
-		)
-		(embedded_fonts no)
-	)
 	(footprint "Texas_DRT_3"
 		(layer "F.Cu")
@@
 		(embedded_fonts no)
 	)
+	(footprint "Crystal_3225_4Pad"
+		(layer "F.Cu")
+		(at 108 130)
+		(descr "3.2 x 2.5 mm 4-pad crystal; verify vendor pad numbering before release")
+		(property "Reference" "Y1"
+			(at 0 0 0)
+			(layer "F.SilkS")
+			(effects
+				(font
+					(size 1.27 1.27)
+				)
+			)
+		)
+		(property "Value" ""
+			(at 0 0 0)
+			(layer "F.Fab")
+			(effects
+				(font
+					(size 1.27 1.27)
+				)
+			)
+		)
+		(property "Datasheet" ""
+			(at 0 0 0)
+			(layer "F.Fab")
+			(hide yes)
+			(effects
+				(font
+					(size 1.27 1.27)
+				)
+			)
+		)
+		(property "Description" ""
+			(at 0 0 0)
+			(layer "F.Fab")
+			(hide yes)
+			(effects
+				(font
+					(size 1.27 1.27)
+				)
+			)
+		)
+		(duplicate_pad_numbers_are_jumpers no)
+		(fp_rect
+			(start -1.6 -1.25)
+			(end 1.6 1.25)
+			(stroke
+				(width 0.12)
+				(type default)
+			)
+			(fill no)
+			(layer "F.SilkS")
+		)
+		(fp_rect
+			(start -1.7 -1.35)
+			(end 1.7 1.35)
+			(stroke
+				(width 0.05)
+				(type default)
+			)
+			(fill no)
+			(layer "F.CrtYd")
+		)
+		(pad "1" smd roundrect
+			(at -1.1 -0.85)
+			(size 1.2 0.9)
+			(layers "F.Cu" "F.Mask" "F.Paste")
+			(roundrect_rratio 0.2)
+			(net "/STORAGE/BRIDGE_XI")
+		)
+		(pad "2" smd roundrect
+			(at -1.1 0.85)
+			(size 1.2 0.9)
+			(layers "F.Cu" "F.Mask" "F.Paste")
+			(roundrect_rratio 0.2)
+			(net "/STORAGE/BRIDGE_VSSOSC")
+		)
+		(pad "3" smd roundrect
+			(at 1.1 0.85)
+			(size 1.2 0.9)
+			(layers "F.Cu" "F.Mask" "F.Paste")
+			(roundrect_rratio 0.2)
+			(net "/STORAGE/BRIDGE_XO")
+		)
+		(pad "4" smd roundrect
+			(at 1.1 -0.85)
+			(size 1.2 0.9)
+			(layers "F.Cu" "F.Mask" "F.Paste")
+			(roundrect_rratio 0.2)
+			(net "/STORAGE/BRIDGE_VSSOSC")
+		)
+		(embedded_fonts no)
+	)
 	(footprint "C_1206_3216Metric"
 		(layer "F.Cu")
@@
 	(segment
 		(start 124 131.5)
-		(end 124 129)
+		(end 124 126)
 		(width 0.1321)
 		(layer "B.Cu")
@@
 	)
 	(segment
-		(start 124 129)
-		(end 107.15 129)
+		(start 106.9 126)
+		(end 106.9 129.15)
 		(width 0.1321)
 		(layer "B.Cu")
@@
 	)
 	(segment
-		(start 107.15 129)
-		(end 107.15 131.1)
+		(start 124 126)
+		(end 106.9 126)
 		(width 0.1321)
 		(layer "B.Cu")
@@
 	(segment
 		(start 122.5 133.5)
-		(end 122.5 130.5)
+		(end 110 133.5)
 		(width 0.1321)
 		(layer "F.Cu")
@@
 	)
 	(segment
-		(start 122.5 135.5)
-		(end 122.5 133.5)
+		(start 110 129.15)
+		(end 109.1 129.15)
 		(width 0.1321)
 		(layer "F.Cu")
 		(net "/STORAGE/BRIDGE_VSSOSC")
 	)
-	(via
-		(at 122.5 130.5)
-		(size 0.5)
-		(drill 0.3)
-		(layers "F.Cu" "B.Cu")
-		(net "/STORAGE/BRIDGE_VSSOSC")
-	)
 	(segment
-		(start 108.85 130)
-		(end 108.85 131.1)
-		(width 0.1321)
-		(layer "B.Cu")
-		(net "/STORAGE/BRIDGE_VSSOSC")
-	)
-	(segment
-		(start 122.5 130)
-		(end 108.85 130)
+		(start 122.5 135.5)
+		(end 122.5 133.5)
 		(width 0.1321)
-		(layer "B.Cu")
+		(layer "F.Cu")
 		(net "/STORAGE/BRIDGE_VSSOSC")
 	)
 	(segment
-		(start 122.5 130.5)
-		(end 122.5 130)
+		(start 110 133.5)
+		(end 110 129.15)
 		(width 0.1321)
-		(layer "B.Cu")
+		(layer "F.Cu")
 		(net "/STORAGE/BRIDGE_VSSOSC")
 	)
 	(segment
-		(start 122 135.5)
-		(end 122 132.5)
+		(start 122 132.5)
+		(end 122 129.5)
 		(width 0.1321)
 		(layer "F.Cu")
@@
 	)
 	(segment
-		(start 122 132.5)
-		(end 122 129.5)
+		(start 122 135.5)
+		(end 122 132.5)
 		(width 0.1321)
 		(layer "F.Cu")
@@
 	)
 	(segment
-		(start 108.85 131)
-		(end 108.85 128.9)
+		(start 122 129.5)
+		(end 122 131.5)
 		(width 0.1321)
 		(layer "B.Cu")
@@
 	)
 	(segment
-		(start 122 129.5)
-		(end 122 131)
+		(start 122 131.5)
+		(end 109.1 131.5)
 		(width 0.1321)
 		(layer "B.Cu")
@@
 	)
 	(segment
-		(start 122 131)
-		(end 108.85 131)
+		(start 109.1 131.5)
+		(end 109.1 130.85)
 		(width 0.1321)
 		(layer "B.Cu")

Commit message: phase24 reject mixed clock escape
Routing:
- net /STORAGE/BRIDGE_XI: track 29.9 -> 38.8 mm
- net /STORAGE/BRIDGE_XO: track 21.6 -> 16.4 mm
Changed lines of the file:
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@@
 		(embedded_fonts no)
 	)
-	(footprint "Crystal_3225_4Pad"
-		(layer "F.Cu")
-		(at 108 130)
-		(descr "3.2 x 2.5 mm 4-pad crystal; verify vendor pad numbering before release")
-		(property "Reference" "Y1"
-			(at 0 0 0)
-			(layer "F.SilkS")
-			(effects
-				(font
-					(size 1.27 1.27)
-				)
-			)
-		)
-		(property "Value" ""
-			(at 0 0 0)
-			(layer "F.Fab")
-			(effects
-				(font
-					(size 1.27 1.27)
-				)
-			)
-		)
-		(property "Datasheet" ""
-			(at 0 0 0)
-			(layer "F.Fab")
-			(hide yes)
-			(effects
-				(font
-					(size 1.27 1.27)
-				)
-			)
-		)
-		(property "Description" ""
-			(at 0 0 0)
-			(layer "F.Fab")
-			(hide yes)
-			(effects
-				(font
-					(size 1.27 1.27)
-				)
-			)
-		)
-		(duplicate_pad_numbers_are_jumpers no)
-		(fp_rect
-			(start -1.6 -1.25)
-			(end 1.6 1.25)
-			(stroke
-				(width 0.12)
-				(type default)
-			)
-			(fill no)
-			(layer "F.SilkS")
-		)
-		(fp_rect
-			(start -1.7 -1.35)
-			(end 1.7 1.35)
-			(stroke
-				(width 0.05)
-				(type default)
-			)
-			(fill no)
-			(layer "F.CrtYd")
-		)
-		(pad "1" smd roundrect
-			(at -1.1 -0.85)
-			(size 1.2 0.9)
-			(layers "F.Cu" "F.Mask" "F.Paste")
-			(roundrect_rratio 0.2)
-			(net "/STORAGE/BRIDGE_XI")
-		)
-		(pad "2" smd roundrect
-			(at -1.1 0.85)
-			(size 1.2 0.9)
-			(layers "F.Cu" "F.Mask" "F.Paste")
-			(roundrect_rratio 0.2)
-			(net "/STORAGE/BRIDGE_VSSOSC")
-		)
-		(pad "3" smd roundrect
-			(at 1.1 0.85)
-			(size 1.2 0.9)
-			(layers "F.Cu" "F.Mask" "F.Paste")
-			(roundrect_rratio 0.2)
-			(net "/STORAGE/BRIDGE_XO")
-		)
-		(pad "4" smd roundrect
-			(at 1.1 -0.85)
-			(size 1.2 0.9)
-			(layers "F.Cu" "F.Mask" "F.Paste")
-			(roundrect_rratio 0.2)
-			(net "/STORAGE/BRIDGE_VSSOSC")
-		)
-		(embedded_fonts no)
-	)
 	(footprint "C_1206_3216Metric"
 		(layer "F.Cu")
@@
 		(embedded_fonts no)
 	)
+	(footprint "Crystal_3225_4Pad"
+		(layer "F.Cu")
+		(at 108 130)
+		(descr "3.2 x 2.5 mm 4-pad crystal; verify vendor pad numbering before release")
+		(property "Reference" "Y1"
+			(at 0 0 0)
+			(layer "F.SilkS")
+			(effects
+				(font
+					(size 1.27 1.27)
+				)
+			)
+		)
+		(property "Value" ""
+			(at 0 0 0)
+			(layer "F.Fab")
+			(effects
+				(font
+					(size 1.27 1.27)
+				)
+			)
+		)
+		(property "Datasheet" ""
+			(at 0 0 0)
+			(layer "F.Fab")
+			(hide yes)
+			(effects
+				(font
+					(size 1.27 1.27)
+				)
+			)
+		)
+		(property "Description" ""
+			(at 0 0 0)
+			(layer "F.Fab")
+			(hide yes)
+			(effects
+				(font
+					(size 1.27 1.27)
+				)
+			)
+		)
+		(duplicate_pad_numbers_are_jumpers no)
+		(fp_rect
+			(start -1.6 -1.25)
+			(end 1.6 1.25)
+			(stroke
+				(width 0.12)
+				(type default)
+			)
+			(fill no)
+			(layer "F.SilkS")
+		)
+		(fp_rect
+			(start -1.7 -1.35)
+			(end 1.7 1.35)
+			(stroke
+				(width 0.05)
+				(type default)
+			)
+			(fill no)
+			(layer "F.CrtYd")
+		)
+		(pad "1" smd roundrect
+			(at -1.1 -0.85)
+			(size 1.2 0.9)
+			(layers "F.Cu" "F.Mask" "F.Paste")
+			(roundrect_rratio 0.2)
+			(net "/STORAGE/BRIDGE_XI")
+		)
+		(pad "2" smd roundrect
+			(at -1.1 0.85)
+			(size 1.2 0.9)
+			(layers "F.Cu" "F.Mask" "F.Paste")
+			(roundrect_rratio 0.2)
+			(net "/STORAGE/BRIDGE_VSSOSC")
+		)
+		(pad "3" smd roundrect
+			(at 1.1 0.85)
+			(size 1.2 0.9)
+			(layers "F.Cu" "F.Mask" "F.Paste")
+			(roundrect_rratio 0.2)
+			(net "/STORAGE/BRIDGE_XO")
+		)
+		(pad "4" smd roundrect
+			(at 1.1 -0.85)
+			(size 1.2 0.9)
+			(layers "F.Cu" "F.Mask" "F.Paste")
+			(roundrect_rratio 0.2)
+			(net "/STORAGE/BRIDGE_VSSOSC")
+		)
+		(embedded_fonts no)
+	)
 	(footprint "TVS_SMBJ18A_DO214AA"
 		(layer "F.Cu")
@@
 	(segment
 		(start 123 134.5)
-		(end 124 131.5)
+		(end 128 134.5)
 		(width 0.1321)
 		(layer "F.Cu")
@@
 	)
 	(via
-		(at 124 131.5)
+		(at 128 134.5)
 		(size 0.5)
 		(drill 0.3)
@@
 	)
 	(segment
-		(start 124 131.5)
-		(end 124 126)
-		(width 0.1321)
-		(layer "B.Cu")
-		(net "/STORAGE/BRIDGE_XI")
-	)
-	(segment
 		(start 106.9 126)
 		(end 106.9 129.15)
@@
 	)
 	(segment
-		(start 124 126)
+		(start 128 126)
 		(end 106.9 126)
 		(width 0.1321)
@@
 	)
 	(segment
-		(start 122.5 133.5)
-		(end 110 133.5)
+		(start 128 134.5)
+		(end 128 126)
 		(width 0.1321)
-		(layer "F.Cu")
-		(net "/STORAGE/BRIDGE_VSSOSC")
+		(layer "B.Cu")
+		(net "/STORAGE/BRIDGE_XI")
 	)
 	(segment
@@
 	)
 	(segment
-		(start 122 132.5)
-		(end 122 129.5)
+		(start 122.5 133.5)
+		(end 110 133.5)
+		(width 0.1321)
+		(layer "F.Cu")
+		(net "/STORAGE/BRIDGE_VSSOSC")
+	)
+	(segment
+		(start 122 134)
+		(end 119 132.5)
 		(width 0.1321)
 		(layer "F.Cu")
@@
 	(segment
 		(start 122 135.5)
-		(end 122 132.5)
+		(end 122 134)
 		(width 0.1321)
 		(layer "F.Cu")
@@
 	)
 	(via
-		(at 122 129.5)
+		(at 119 132.5)
 		(size 0.5)
 		(drill 0.3)
@@
 	)
 	(segment
-		(start 122 129.5)
-		(end 122 131.5)
+		(start 119 131.5)
+		(end 109.1 131.5)
 		(width 0.1321)
 		(layer "B.Cu")
@@
 	)
 	(segment
-		(start 122 131.5)
-		(end 109.1 131.5)
+		(start 119 132.5)
+		(end 119 131.5)
 		(width 0.1321)
 		(layer "B.Cu")
