File: pisxme/reva-clean/PHASE24_SUPPORT_BRANCH_ASTAR.kicad_pcb (KiCad board)
At the start: 6 copper layers, 300 x 180 mm, 97 parts, among them J1 74221-101LF, J2 A70-112-331N126, J3 JAE SM3ZS067U410ABR1000 B-key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, J4 Amphenol 10171746-00021LF USB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, J5 0039300020, J6 0039300020, J7 Raspberry-Pi-5-Compute-Module, Q1 CSD19536KCS, Q2 CSD19536KCS, U1 LM74700QDBVRQ1, U2 LM74700QDBVRQ1, U3 TPSM63606RDLR, U4 TPSM63606RDLR, U5 TPSM63606RDLR, U6 TPD4EUSB30, U7 TUSB9261IPVP, U8 Texas_DRT_3, U9 TPD4EUSB30

Commit message: phase24 reject passive placement sweep
Parts:
- moved C42 25.7 mm to (108.0, 145.0)
- moved C43 25.7 mm to (120.0, 145.0)
- moved R23 25.7 mm to (114.0, 145.0)
Routing:
- net /STORAGE/BRIDGE_XI: track 58.4 -> 84.4 mm
- net /STORAGE/BRIDGE_XO: track 60.0 -> 82.0 mm
- net /STORAGE/BRIDGE_VSSOSC: track 106.1 -> 89.6 mm

Commit message: phase24 reject graph anchor fanout
Parts:
- moved C42 25.7 mm to (102.0, 120.0)
- moved C43 25.7 mm to (114.0, 120.0)
- moved R23 25.7 mm to (108.0, 120.0)
Routing:
- net /STORAGE/BRIDGE_XI: track 84.4 -> 54.9 mm
- net /STORAGE/BRIDGE_XO: track 82.0 -> 58.0 mm
- net /STORAGE/BRIDGE_VSSOSC: track 89.6 -> 77.1 mm
