File: pisxme/reva-clean/PHASE24_CLOCK_OBSTACLE_REGEN.kicad_pcb (KiCad board)
At the start: 6 copper layers, 300 x 180 mm, 92 parts, among them J1 74221-101LF, J2 A70-112-331N126, J3 JAE SM3ZS067U410ABR1000 B-key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, J4 Amphenol 10171746-00021LF USB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, J5 0039300020, J6 0039300020, J7 Raspberry-Pi-5-Compute-Module, Q1 CSD19536KCS, Q2 CSD19536KCS, U1 LM74700QDBVRQ1, U2 LM74700QDBVRQ1, U3 TPSM63606RDLR, U4 TPSM63606RDLR, U5 TPSM63606RDLR, U6 TPD4EUSB30, U7 TUSB9261IPVP, U8 Texas_DRT_3, U9 TPD4EUSB30

Commit message: phase24 harden U5 negative controls
Parts:
- moved Y1 21.5 mm to (100.0, 150.0)
- moved C42 20.6 mm to (96.0, 146.0)
- moved C43 20.6 mm to (96.0, 154.0)
- moved R23 20.6 mm to (96.0, 150.0)
Routing:
- net /STORAGE/BRIDGE_XI: track 50.6 -> 72.4 mm
- net /STORAGE/BRIDGE_VSSOSC: track 63.8 -> 84.2 mm
- net /STORAGE/BRIDGE_XO: track 44.4 -> 53.5 mm, vias 4 -> 5
