File: pisxme/reva-clean/PHASE24_MACRO_ETH_SOUTH.kicad_pcb (KiCad board)
At the start: 6 copper layers, 300 x 180 mm, 92 parts, among them J1 74221-101LF, J2 A70-112-331N126, J3 JAE SM3ZS067U410ABR1000 B-key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, J4 Amphenol 10171746-00021LF USB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, J5 0039300020, J6 0039300020, J7 Raspberry-Pi-5-Compute-Module, Q1 CSD19536KCS, Q2 CSD19536KCS, U1 LM74700QDBVRQ1, U2 LM74700QDBVRQ1, U3 TPSM63606RDLR, U4 TPSM63606RDLR, U5 TPSM63606RDLR, U6 TPD4EUSB30, U7 TUSB9261IPVP, U8 Texas_DRT_3, U9 TPD4EUSB30

Commit message: phase24 correct macro floorplan authority
Parts:
- moved U6 45.3 mm to (42.0, 88.0)
- moved U9 35.4 mm to (48.0, 88.0)
- moved U8 20.0 mm to (58.0, 100.0)
Changed lines of the file:
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@@
 	(footprint "Package_SON:USON-10_2.5x1.0mm_P0.5mm"
 		(layer "F.Cu")
-		(at 75.1 65.215 -90)
+		(at 48 88 -90)
 		(descr "USON-10 2.5x1.0mm_ Pitch 0.5mm http://www.ti.com/lit/ds/symlink/tpd4e02b04.pdf")
 		(tags "USON-10 2.5x1.0mm Pitch 0.5mm")
@@
 	(footprint "Package_SON:USON-10_2.5x1.0mm_P0.5mm"
 		(layer "F.Cu")
-		(at 81.1 65.215 -90)
+		(at 42 88 -90)
 		(descr "USON-10 2.5x1.0mm_ Pitch 0.5mm http://www.ti.com/lit/ds/symlink/tpd4e02b04.pdf")
 		(tags "USON-10 2.5x1.0mm Pitch 0.5mm")
@@
 	(footprint "Texas_DRT_3"
 		(layer "F.Cu")
-		(at 38 100 90)
+		(at 58 100 90)
 		(descr "Texas Instruments DRT-3 1x0.8mm, 0.7mm pitch; TI TPD2EUSB30 datasheet; KiCad maintained footprint")
 		(tags "DRT-3 1x0.8mm Pitch 0.7mm")
