File: pisxme/reva-clean/PHASE24_ETHERNET_SUPPORT_FIXTURE.kicad_sch (KiCad schematic)
At the start: 15 parts, among them J2 A70-112-331N126, U6 TPD4EUSB30DQAR, U9 TPD4EUSB30DQAR, X6 ETHERNET_Contract

Commit message: phase24: source ethernet support passives
Parts:
- C48, C49, C50, C51: footprint PiSXMeRevAClean:C_0402_1005Metric -> PiSXMeRevAClean:C_0603_1608Metric; MPN PROVISIONAL_NOT_PROCUREMENT_AUTHORITY -> GRM188R72A223KAC4J
- C52: MPN PROVISIONAL_NOT_PROCUREMENT_AUTHORITY -> 1206GC102KAT2A
- R26, R27, R28, R29: MPN PROVISIONAL_NOT_PROCUREMENT_AUTHORITY -> CRCW040275R0FKEDC
- R30, R31: MPN PROVISIONAL_NOT_PROCUREMENT_AUTHORITY -> RK73G1ETTP4700D
Changed lines of the file:
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@@
  (property "Reference" "C48" (at 108 46 0) (effects (font (size 1 1))))
  (property "Value" "22nF 100V" (at 108 54 0) (effects (font (size 1 1))))
- (property "MPN" "PROVISIONAL_NOT_PROCUREMENT_AUTHORITY" (at 108 50 0) (effects (font (size 1 1)) (hide yes)))
- (property "Footprint" "PiSXMeRevAClean:C_0402_1005Metric" (at 108 50 0) (effects (font (size 1 1)) (hide yes)))
+ (property "MPN" "GRM188R72A223KAC4J" (at 108 50 0) (effects (font (size 1 1)) (hide yes)))
+ (property "Footprint" "PiSXMeRevAClean:C_0603_1608Metric" (at 108 50 0) (effects (font (size 1 1)) (hide yes)))
  (pin "1") (pin "2")
  (instances (project "PiSXMe_RevA_Clean" (path "/30000000-0000-0000-0000-000000000000/10000000-0000-0000-0000-000000000006" (reference "C48") (unit 1)))) )
@@
  (property "Reference" "R26" (at 108 56 0) (effects (font (size 1 1))))
  (property "Value" "75R" (at 108 64 0) (effects (font (size 1 1))))
- (property "MPN" "PROVISIONAL_NOT_PROCUREMENT_AUTHORITY" (at 108 60 0) (effects (font (size 1 1)) (hide yes)))
+ (property "MPN" "CRCW040275R0FKEDC" (at 108 60 0) (effects (font (size 1 1)) (hide yes)))
  (property "Footprint" "PiSXMeRevAClean:R_0402_1005Metric" (at 108 60 0) (effects (font (size 1 1)) (hide yes)))
  (pin "1") (pin "2")
@@
  (property "Reference" "C49" (at 116 46 0) (effects (font (size 1 1))))
  (property "Value" "22nF 100V" (at 116 54 0) (effects (font (size 1 1))))
- (property "MPN" "PROVISIONAL_NOT_PROCUREMENT_AUTHORITY" (at 116 50 0) (effects (font (size 1 1)) (hide yes)))
- (property "Footprint" "PiSXMeRevAClean:C_0402_1005Metric" (at 116 50 0) (effects (font (size 1 1)) (hide yes)))
+ (property "MPN" "GRM188R72A223KAC4J" (at 116 50 0) (effects (font (size 1 1)) (hide yes)))
+ (property "Footprint" "PiSXMeRevAClean:C_0603_1608Metric" (at 116 50 0) (effects (font (size 1 1)) (hide yes)))
  (pin "1") (pin "2")
  (instances (project "PiSXMe_RevA_Clean" (path "/30000000-0000-0000-0000-000000000000/10000000-0000-0000-0000-000000000006" (reference "C49") (unit 1)))) )
@@
  (property "Reference" "R27" (at 116 56 0) (effects (font (size 1 1))))
  (property "Value" "75R" (at 116 64 0) (effects (font (size 1 1))))
- (property "MPN" "PROVISIONAL_NOT_PROCUREMENT_AUTHORITY" (at 116 60 0) (effects (font (size 1 1)) (hide yes)))
+ (property "MPN" "CRCW040275R0FKEDC" (at 116 60 0) (effects (font (size 1 1)) (hide yes)))
  (property "Footprint" "PiSXMeRevAClean:R_0402_1005Metric" (at 116 60 0) (effects (font (size 1 1)) (hide yes)))
  (pin "1") (pin "2")
@@
  (property "Reference" "C50" (at 124 46 0) (effects (font (size 1 1))))
  (property "Value" "22nF 100V" (at 124 54 0) (effects (font (size 1 1))))
- (property "MPN" "PROVISIONAL_NOT_PROCUREMENT_AUTHORITY" (at 124 50 0) (effects (font (size 1 1)) (hide yes)))
- (property "Footprint" "PiSXMeRevAClean:C_0402_1005Metric" (at 124 50 0) (effects (font (size 1 1)) (hide yes)))
+ (property "MPN" "GRM188R72A223KAC4J" (at 124 50 0) (effects (font (size 1 1)) (hide yes)))
+ (property "Footprint" "PiSXMeRevAClean:C_0603_1608Metric" (at 124 50 0) (effects (font (size 1 1)) (hide yes)))
  (pin "1") (pin "2")
  (instances (project "PiSXMe_RevA_Clean" (path "/30000000-0000-0000-0000-000000000000/10000000-0000-0000-0000-000000000006" (reference "C50") (unit 1)))) )
@@
  (property "Reference" "R28" (at 124 56 0) (effects (font (size 1 1))))
  (property "Value" "75R" (at 124 64 0) (effects (font (size 1 1))))
- (property "MPN" "PROVISIONAL_NOT_PROCUREMENT_AUTHORITY" (at 124 60 0) (effects (font (size 1 1)) (hide yes)))
+ (property "MPN" "CRCW040275R0FKEDC" (at 124 60 0) (effects (font (size 1 1)) (hide yes)))
  (property "Footprint" "PiSXMeRevAClean:R_0402_1005Metric" (at 124 60 0) (effects (font (size 1 1)) (hide yes)))
  (pin "1") (pin "2")
@@
  (property "Reference" "C51" (at 132 46 0) (effects (font (size 1 1))))
  (property "Value" "22nF 100V" (at 132 54 0) (effects (font (size 1 1))))
- (property "MPN" "PROVISIONAL_NOT_PROCUREMENT_AUTHORITY" (at 132 50 0) (effects (font (size 1 1)) (hide yes)))
- (property "Footprint" "PiSXMeRevAClean:C_0402_1005Metric" (at 132 50 0) (effects (font (size 1 1)) (hide yes)))
+ (property "MPN" "GRM188R72A223KAC4J" (at 132 50 0) (effects (font (size 1 1)) (hide yes)))
+ (property "Footprint" "PiSXMeRevAClean:C_0603_1608Metric" (at 132 50 0) (effects (font (size 1 1)) (hide yes)))
  (pin "1") (pin "2")
  (instances (project "PiSXMe_RevA_Clean" (path "/30000000-0000-0000-0000-000000000000/10000000-0000-0000-0000-000000000006" (reference "C51") (unit 1)))) )
@@
  (property "Reference" "R29" (at 132 56 0) (effects (font (size 1 1))))
  (property "Value" "75R" (at 132 64 0) (effects (font (size 1 1))))
- (property "MPN" "PROVISIONAL_NOT_PROCUREMENT_AUTHORITY" (at 132 60 0) (effects (font (size 1 1)) (hide yes)))
+ (property "MPN" "CRCW040275R0FKEDC" (at 132 60 0) (effects (font (size 1 1)) (hide yes)))
  (property "Footprint" "PiSXMeRevAClean:R_0402_1005Metric" (at 132 60 0) (effects (font (size 1 1)) (hide yes)))
  (pin "1") (pin "2")
@@
  (property "Reference" "C52" (at 108 71 0) (effects (font (size 1 1))))
  (property "Value" "1nF 2kV" (at 108 79 0) (effects (font (size 1 1))))
- (property "MPN" "PROVISIONAL_NOT_PROCUREMENT_AUTHORITY" (at 108 75 0) (effects (font (size 1 1)) (hide yes)))
+ (property "MPN" "1206GC102KAT2A" (at 108 75 0) (effects (font (size 1 1)) (hide yes)))
  (property "Footprint" "PiSXMeRevAClean:C_1206_3216Metric" (at 108 75 0) (effects (font (size 1 1)) (hide yes)))
  (pin "1") (pin "2")
@@
  (property "Reference" "R30" (at 145 46 0) (effects (font (size 1 1))))
  (property "Value" "470R" (at 145 54 0) (effects (font (size 1 1))))
- (property "MPN" "PROVISIONAL_NOT_PROCUREMENT_AUTHORITY" (at 145 50 0) (effects (font (size 1 1)) (hide yes)))
+ (property "MPN" "RK73G1ETTP4700D" (at 145 50 0) (effects (font (size 1 1)) (hide yes)))
  (property "Footprint" "PiSXMeRevAClean:R_0402_1005Metric" (at 145 50 0) (effects (font (size 1 1)) (hide yes)))
  (pin "1") (pin "2")
@@
  (property "Reference" "R31" (at 155 46 0) (effects (font (size 1 1))))
  (property "Value" "470R" (at 155 54 0) (effects (font (size 1 1))))
- (property "MPN" "PROVISIONAL_NOT_PROCUREMENT_AUTHORITY" (at 155 50 0) (effects (font (size 1 1)) (hide yes)))
+ (property "MPN" "RK73G1ETTP4700D" (at 155 50 0) (effects (font (size 1 1)) (hide yes)))
  (property "Footprint" "PiSXMeRevAClean:R_0402_1005Metric" (at 155 50 0) (effects (font (size 1 1)) (hide yes)))
  (pin "1") (pin "2")
