File: pisxme/reva-clean/PHASE24_ETHERNET_LOCAL_ESCAPE_PROBE.kicad_pcb (KiCad board)
At the start: 6 copper layers, 300 x 180 mm, 92 parts, among them J1 74221-101LF, J2 A70-112-331N126, J3 JAE SM3ZS067U410ABR1000 B-key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, J4 Amphenol 10171746-00021LF USB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, J5 0039300020, J6 0039300020, J7 Raspberry-Pi-5-Compute-Module, Q1 CSD19536KCS, Q2 CSD19536KCS, U1 LM74700QDBVRQ1, U2 LM74700QDBVRQ1, U3 TPSM63606RDLR, U4 TPSM63606RDLR, U5 TPSM63606RDLR, U6 TPD4EUSB30, U7 TUSB9261IPVP, U8 Texas_DRT_3, U9 TPD4EUSB30

Commit message: phase24: test wider Ethernet staging escape
Parts:
- moved U6 11.3 mm to (12.0, 112.0)
- moved U9 10.0 mm to (20.0, 112.0)
Routing:
- net CM5_GBE_TD0_P: track 20.4 -> 30.8 mm
- net CM5_GBE_TD0_N: track 18.5 -> 28.9 mm
- net CM5_GBE_TD1_N: track 18.4 -> 28.8 mm
- net CM5_GBE_TD1_P: track 20.3 -> 30.6 mm
- net CM5_GBE_TD2_P: track 12.0 -> 21.7 mm
- net CM5_GBE_TD2_N: track 10.1 -> 19.8 mm
- net CM5_GBE_TD3_N: track 9.96 -> 19.6 mm
- net CM5_GBE_TD3_P: track 11.8 -> 21.5 mm
Changed lines of the file:
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@@
 	(footprint "Package_SON:USON-10_2.5x1.0mm_P0.5mm"
 		(layer "F.Cu")
-		(at 26 104)
+		(at 20 112)
 		(descr "USON-10 2.5x1.0mm_ Pitch 0.5mm http://www.ti.com/lit/ds/symlink/tpd4e02b04.pdf")
 		(tags "USON-10 2.5x1.0mm Pitch 0.5mm")
@@
 	(footprint "Package_SON:USON-10_2.5x1.0mm_P0.5mm"
 		(layer "F.Cu")
-		(at 20 104)
+		(at 12 112)
 		(descr "USON-10 2.5x1.0mm_ Pitch 0.5mm http://www.ti.com/lit/ds/symlink/tpd4e02b04.pdf")
 		(tags "USON-10 2.5x1.0mm Pitch 0.5mm")
@@
 	)
 	(segment
-		(start 26.385 105)
-		(end 26.385 103)
+		(start 20.385 113)
+		(end 20.385 111)
 		(width 0.127)
 		(layer "F.Cu")
@@
 	(segment
 		(start 32.96 100.7)
-		(end 26.385 105)
+		(end 20.385 113)
 		(width 0.127)
 		(layer "F.Cu")
@@
 	)
 	(segment
-		(start 26.385 105)
-		(end 25.615 103)
+		(start 20.385 113)
+		(end 19.615 111)
 		(width 0.127)
 		(layer "F.Cu")
@@
 	)
 	(segment
-		(start 26.385 104.5)
-		(end 26.385 103.5)
+		(start 20.385 112.5)
+		(end 19.615 111.5)
 		(width 0.127)
 		(layer "F.Cu")
@@
 	)
 	(segment
-		(start 32.96 100.3)
-		(end 26.385 104.5)
+		(start 20.385 112.5)
+		(end 20.385 111.5)
 		(width 0.127)
 		(layer "F.Cu")
@@
 	)
 	(segment
-		(start 26.385 104.5)
-		(end 25.615 103.5)
+		(start 32.96 100.3)
+		(end 20.385 112.5)
 		(width 0.127)
 		(layer "F.Cu")
@@
 	(segment
 		(start 32.96 99.5)
-		(end 26.385 103.5)
+		(end 20.385 111.5)
 		(width 0.127)
 		(layer "F.Cu")
@@
 	)
 	(segment
-		(start 26.385 103.5)
-		(end 26.385 104.5)
+		(start 20.385 111.5)
+		(end 19.615 112.5)
 		(width 0.127)
 		(layer "F.Cu")
@@
 	)
 	(segment
-		(start 26.385 103.5)
-		(end 25.615 104.5)
+		(start 20.385 111.5)
+		(end 20.385 112.5)
 		(width 0.127)
 		(layer "F.Cu")
@@
 	)
 	(segment
-		(start 26.385 103)
-		(end 26.385 105)
+		(start 20.385 111)
+		(end 20.385 113)
 		(width 0.127)
 		(layer "F.Cu")
@@
 	)
 	(segment
-		(start 26.385 103)
-		(end 25.615 105)
+		(start 32.96 99.1)
+		(end 20.385 111)
 		(width 0.127)
 		(layer "F.Cu")
@@
 	)
 	(segment
-		(start 32.96 99.1)
-		(end 26.385 103)
+		(start 20.385 111)
+		(end 19.615 113)
 		(width 0.127)
 		(layer "F.Cu")
@@
 	)
 	(segment
-		(start 20.385 105)
-		(end 19.615 103)
+		(start 36.04 100.7)
+		(end 12.385 113)
 		(width 0.127)
 		(layer "F.Cu")
@@
 	)
 	(segment
-		(start 36.04 100.7)
-		(end 20.385 105)
+		(start 12.385 113)
+		(end 11.615 111)
 		(width 0.127)
 		(layer "F.Cu")
@@
 	)
 	(segment
-		(start 20.385 105)
-		(end 20.385 103)
+		(start 12.385 113)
+		(end 12.385 111)
 		(width 0.127)
 		(layer "F.Cu")
@@
 	)
 	(segment
-		(start 36.04 100.3)
-		(end 20.385 104.5)
+		(start 12.385 112.5)
+		(end 11.615 111.5)
 		(width 0.127)
 		(layer "F.Cu")
@@
 	)
 	(segment
-		(start 20.385 104.5)
-		(end 19.615 103.5)
+		(start 12.385 112.5)
+		(end 12.385 111.5)
 		(width 0.127)
 		(layer "F.Cu")
@@
 	)
 	(segment
-		(start 20.385 104.5)
-		(end 20.385 103.5)
+		(start 36.04 100.3)
+		(end 12.385 112.5)
 		(width 0.127)
 		(layer "F.Cu")
@@
 	)
 	(segment
-		(start 20.385 103.5)
-		(end 20.385 104.5)
+		(start 36.04 99.5)
+		(end 12.385 111.5)
 		(width 0.127)
 		(layer "F.Cu")
@@
 	)
 	(segment
-		(start 36.04 99.5)
-		(end 20.385 103.5)
+		(start 12.385 111.5)
+		(end 12.385 112.5)
 		(width 0.127)
 		(layer "F.Cu")
@@
 	)
 	(segment
-		(start 20.385 103.5)
-		(end 19.615 104.5)
+		(start 12.385 111.5)
+		(end 11.615 112.5)
 		(width 0.127)
 		(layer "F.Cu")
@@
 	)
 	(segment
-		(start 20.385 103)
-		(end 20.385 105)
+		(start 12.385 111)
+		(end 11.615 113)
 		(width 0.127)
 		(layer "F.Cu")
@@
 	)
 	(segment
-		(start 20.385 103)
-		(end 19.615 105)
+		(start 12.385 111)
+		(end 12.385 113)
 		(width 0.127)
 		(layer "F.Cu")
@@
 	(segment
 		(start 36.04 99.1)
-		(end 20.385 103)
+		(end 12.385 111)
 		(width 0.127)
 		(layer "F.Cu")
