File: pisxme/reva-clean/PHASE24_MACRO_FRESH_ETH_EAST_STORAGE_NORTH.kicad_pcb (KiCad board)
At the start: 6 copper layers, 300 x 180 mm, 92 parts, among them J1 74221-101LF, J2 A70-112-331N126, J3 JAE SM3ZS067U410ABR1000 B-key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, J4 Amphenol 10171746-00021LF USB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, J5 0039300020, J6 0039300020, J7 Raspberry-Pi-5-Compute-Module, Q1 CSD19536KCS, Q2 CSD19536KCS, U1 LM74700QDBVRQ1, U2 LM74700QDBVRQ1, U3 TPSM63606RDLR, U4 TPSM63606RDLR, U5 TPSM63606RDLR, U6 TPD4EUSB30, U7 TUSB9261IPVP, U8 Texas_DRT_3, U9 TPD4EUSB30

Commit message: phase24: complete current-basis macro floorplan discriminator
Parts:
- added C48: C_0603_1608Metric, C_0603_1608Metric, B.Cu at (72.0, 45.0)
- added C49: C_0603_1608Metric, C_0603_1608Metric, B.Cu at (93.0, 45.0)
- added C50: C_0603_1608Metric, C_0603_1608Metric, B.Cu at (62.0, 45.0)
- added C51: C_0603_1608Metric, C_0603_1608Metric, B.Cu at (57.0, 45.0)
- added C52: , C_1206_3216Metric, B.Cu at (77.0, 40.0)
- added R26: R_0402_1005Metric, R_0402_1005Metric, B.Cu at (72.0, 40.0)
- added R27: R_0402_1005Metric, R_0402_1005Metric, B.Cu at (93.0, 40.0)
- added R28: R_0402_1005Metric, R_0402_1005Metric, B.Cu at (62.0, 40.0)
- added R29: R_0402_1005Metric, R_0402_1005Metric, B.Cu at (57.0, 40.0)
- C16, C17, C19: moved to B.Cu
- moved C16 9.22 mm to (95.0, 118.0)
- moved C17 7.28 mm to (101.0, 118.0)
- moved C19 3.61 mm to (107.0, 118.0)
Connections:
- J2 pad 15: /ETHERNET/GBE_LED_Y_A -> /ETHERNET/ETH_POWER
- J2 pad 17: /ETHERNET/GBE_LED_G_A -> /ETHERNET/ETH_POWER
- U7 pad 30: (no net) -> /STORAGE/BRIDGE_3V3
- U7 pad 31: (no net) -> /STORAGE/BRIDGE_3V3
Routing:
- net /REGULATORS/BRIDGE_1V1: track 369.0 -> 132.0 mm, vias 19 -> 20
- net /POWER_INPUT/FUSED_12V_A: track 75.5 -> 205.8 mm, vias 1 -> 2
- net /CORE_CM5/POWER_GND: track 83.6 -> 0.00 mm, vias 1 -> 0
- net ETH_CT_COMMON: track 70.8 -> 0.00 mm
- net /ETHERNET/ETH_CT_COMMON: track 0.00 -> 70.8 mm
- net /STORAGE/BRIDGE_SATA_TX_P: track 64.5 -> 9.26 mm
- net POWER_GND: track 261.7 -> 294.7 mm, vias 31 -> 30
- net 12V_PROTECTED: track 250.5 -> 278.3 mm
- net /REGULATORS/FB_CM5_5V: track 0.00 -> 17.0 mm
- net CM5_GBE_TD3_P: track 63.5 -> 80.0 mm, vias 0 -> 1
- net /REGULATORS/BRIDGE_3V3: track 37.1 -> 22.0 mm, vias 3 -> 0
- net CM5_GBE_TD1_P: track 69.7 -> 82.4 mm, vias 0 -> 1
- net /STORAGE/BRIDGE_SATA_RX_P: track 35.0 -> 23.0 mm
- net CM5_GBE_TD3_N: track 64.2 -> 75.6 mm, vias 0 -> 2
- net CM5_GBE_TD2_P: track 65.7 -> 76.9 mm
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- added copper zone on In3.Cu, net /POWER_INPUT/12V_IN_B
- added copper zone on In3.Cu, net /POWER_INPUT/FUSED_12V_B
- added copper zone on In2.Cu, net /REGULATORS/BRIDGE_1V1
- removed copper zone on In3.Cu, net 12V_PROTECTED
