File: pisxme/reva-clean/PHASE24_U7_STORAGE_3V3_PAD24_CURRENT.kicad_pcb (KiCad board)
At the start: 6 copper layers, 300 x 180 mm, 101 parts, among them J1 74221-101LF, J2 A70-112-331N126, J3 JAE SM3ZS067U410ABR1000 B-key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, J4 Amphenol 10171746-00021LF USB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, J5 0039300020, J6 0039300020, J7 Raspberry-Pi-5-Compute-Module, Q1 CSD19536KCS, Q2 CSD19536KCS, U1 LM74700QDBVRQ1, U2 LM74700QDBVRQ1, U3 TPSM63606RDLR, U4 TPSM63606RDLR, U5 TPSM63606RDLR, U6 TPD4EUSB30, U7 TUSB9261IPVP, U8 Texas_DRT_3, U9 TPD4EUSB30

Commit message: phase24: complete current-basis macro floorplan discriminator
Parts:
- moved U7 41.0 mm to (120.0, 140.0)
- moved Y1 24.7 mm to (108.0, 130.0)
- moved J3 23.9 mm to (145.0, 125.0)
- moved C42 23.8 mm to (101.0, 126.0)
- moved C43 23.8 mm to (101.0, 134.0)
- moved R23 23.8 mm to (101.0, 130.0)
Changed lines of the file:
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@@
 	(footprint "C_0402_1005Metric"
 		(layer "F.Cu")
-		(at 78 120)
+		(at 101 126)
 		(property "Reference" "C42"
 			(at 0 -1.1 0)
@@
 	(footprint "TUSB9261IPVP_HTQFP64"
 		(layer "F.Cu")
-		(at 90 112 180)
+		(at 120 140 180)
 		(descr "TUSB9261IPVP; package outline is datasheet-derived and requires final fab-library review")
 		(property "Reference" "U7"
@@
 	(footprint "C_0402_1005Metric"
 		(layer "F.Cu")
-		(at 78 128)
+		(at 101 134)
 		(property "Reference" "C43"
 			(at 0 -1.1 0)
@@
 	(footprint "Crystal_3225_4Pad"
 		(layer "F.Cu")
-		(at 84 124)
+		(at 108 130)
 		(descr "3.2 x 2.5 mm 4-pad crystal; verify vendor pad numbering before release")
 		(property "Reference" "Y1"
@@
 	(footprint "R_0402_1005Metric"
 		(layer "F.Cu")
-		(at 78 124)
+		(at 101 130)
 		(descr "IPC-7351 nominal 0402 resistor; 1.00 x 0.50 mm body; clean-project commodity passive")
 		(property "Reference" "R23"
@@
 	(footprint "JAE_SM3ZS067U410ABR1000_BKEY"
 		(layer "F.Cu")
-		(at 125 112 90)
+		(at 145 125 90)
 		(property "Reference" "J3"
 			(at -7.62 -10.287 90)
