File: pisxme/reva-clean/PHASE24_STORAGE_LOCAL_J3_EDGE_MANUAL_MONOTONIC.kicad_pcb (KiCad board)
At the start: 6 copper layers, 300 x 180 mm, 101 parts, among them J1 74221-101LF, J2 A70-112-331N126, J3 JAE SM3ZS067U410ABR1000 B-key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, J4 Amphenol 10171746-00021LF USB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, J5 0039300020, J6 0039300020, J7 Raspberry-Pi-5-Compute-Module, Q1 CSD19536KCS, Q2 CSD19536KCS, U1 LM74700QDBVRQ1, U2 LM74700QDBVRQ1, U3 TPSM63606RDLR, U4 TPSM63606RDLR, U5 TPSM63606RDLR, U6 TPD4EUSB30, U7 TUSB9261IPVP, U8 Texas_DRT_3, U9 TPD4EUSB30

Commit message: phase24: record storage route development boundary
Routing:
- net /CORE_CM5/CM5_USB3_TX_N: track 26.8 -> 29.7 mm
- net /CORE_CM5/CM5_USB3_TX_P: track 27.8 -> 29.8 mm
Changed lines of the file:
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@@
 	)
 	(via
-		(at 82 103.9)
+		(at 72 103.9)
 		(size 0.5)
 		(drill 0.3)
@@
 	)
 	(via
-		(at 72 103.9)
+		(at 82 103.9)
 		(size 0.5)
 		(drill 0.3)
@@
 		(layer "B.Cu")
 		(net "/CORE_CM5/CM5_USB3_RX_N")
-	)
-	(segment
-		(start 83 108.8)
-		(end 83 119)
-		(width 0.15)
-		(layer "F.Cu")
-		(net "/CORE_CM5/CM5_USB3_RX_P")
 	)
 	(segment
@@
 		(net "/CORE_CM5/CM5_USB3_RX_P")
 	)
+	(segment
+		(start 83 108.8)
+		(end 83 119)
+		(width 0.15)
+		(layer "F.Cu")
+		(net "/CORE_CM5/CM5_USB3_RX_P")
+	)
 	(via
-		(at 83 108.8)
+		(at 72 104.8)
 		(size 0.5)
 		(drill 0.3)
@@
 	)
 	(via
-		(at 72 104.8)
+		(at 83 108.8)
 		(size 0.5)
 		(drill 0.3)
@@
 	)
 	(segment
+		(start 70.04 106.3)
+		(end 72 106.3)
+		(width 0.15)
+		(layer "F.Cu")
+		(net "/CORE_CM5/CM5_USB3_TX_N")
+	)
+	(segment
+		(start 85 121.5)
+		(end 85.5 121.5)
+		(width 0.15)
+		(layer "F.Cu")
+		(net "/CORE_CM5/CM5_USB3_TX_N")
+	)
+	(segment
 		(start 80 110.5)
 		(end 80 117)
@@
 	)
 	(segment
-		(start 80 117)
-		(end 85.5 121.5)
+		(start 85 117)
+		(end 85 121.5)
 		(width 0.15)
 		(layer "F.Cu")
@@
 	)
 	(segment
-		(start 70.04 106.3)
-		(end 72 106.3)
+		(start 80 117)
+		(end 85 117)
 		(width 0.15)
 		(layer "F.Cu")
+		(net "/CORE_CM5/CM5_USB3_TX_N")
+	)
+	(via
+		(at 72 106.3)
+		(size 0.5)
+		(drill 0.3)
+		(layers "F.Cu" "B.Cu")
 		(net "/CORE_CM5/CM5_USB3_TX_N")
 	)
@@
 		(net "/CORE_CM5/CM5_USB3_TX_N")
 	)
-	(via
-		(at 72 106.3)
-		(size 0.5)
-		(drill 0.3)
-		(layers "F.Cu" "B.Cu")
+	(segment
+		(start 72 106.3)
+		(end 72 109.5)
+		(width 0.15)
+		(layer "B.Cu")
 		(net "/CORE_CM5/CM5_USB3_TX_N")
 	)
@@
 	)
 	(segment
-		(start 72 106.3)
-		(end 72 109.5)
+		(start 84 122)
+		(end 85.5 122)
 		(width 0.15)
-		(layer "B.Cu")
-		(net "/CORE_CM5/CM5_USB3_TX_N")
+		(layer "F.Cu")
+		(net "/CORE_CM5/CM5_USB3_TX_P")
 	)
 	(segment
-		(start 81.5 119)
-		(end 85.5 122)
+		(start 84 119)
+		(end 84 122)
 		(width 0.15)
 		(layer "F.Cu")
@@
 		(net "/CORE_CM5/CM5_USB3_TX_P")
 	)
+	(segment
+		(start 81.5 119)
+		(end 84 119)
+		(width 0.15)
+		(layer "F.Cu")
+		(net "/CORE_CM5/CM5_USB3_TX_P")
+	)
 	(via
-		(at 81.5 112)
+		(at 73 106.7)
 		(size 0.5)
 		(drill 0.3)
@@
 	)
 	(via
-		(at 73 106.7)
+		(at 81.5 112)
 		(size 0.5)
 		(drill 0.3)
