File: pisxme/reva-clean/PHASE24_DUAL_MODE_STORAGE_USB3_ISOLATED.kicad_pcb (KiCad board)
At the start: 6 copper layers, 300 x 180 mm, 5 parts, among them J7 Raspberry-Pi-5-Compute-Module

Commit message: phase24 order storage usb3 bridge vias
Routing:
- net JMS_USB3_TXN: track 100.6 -> 48.6 mm
- net JMS_USB3_TXP: track 86.0 -> 40.0 mm
Changed lines of the file:
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@@
+	)
+	(segment
+		(start 70.04 103.9)
+		(end 74 100)
+		(width 0.2)
+		(layer "F.Cu")
+		(net "/CORE_CM5/CM5_USB3_RX_N")
+	)
+	(segment
+		(start 156 152.8)
+		(end 163.5 152.8)
+		(width 0.2)
+		(layer "F.Cu")
+		(net "/CORE_CM5/CM5_USB3_RX_N")
 	)
 	(segment
@@
 		(net "/CORE_CM5/CM5_USB3_RX_N")
 	)
-	(segment
-		(start 70.04 103.9)
-		(end 74 100)
-		(width 0.2)
-		(layer "F.Cu")
-		(net "/CORE_CM5/CM5_USB3_RX_N")
-	)
-	(segment
-		(start 156 152.8)
-		(end 163.5 152.8)
-		(width 0.2)
-		(layer "F.Cu")
-		(net "/CORE_CM5/CM5_USB3_RX_N")
-	)
 	(via
 		(at 74 100)
@@
 	)
 	(segment
+		(start 158 152.6)
+		(end 158 152.4)
+		(width 0.2)
+		(layer "F.Cu")
+		(net "/CORE_CM5/CM5_USB3_RX_P")
+	)
+	(segment
 		(start 70.04 104.3)
 		(end 78 102)
@@
 		(net "/CORE_CM5/CM5_USB3_RX_P")
 	)
-	(segment
-		(start 158 152.6)
-		(end 158 152.4)
-		(width 0.2)
-		(layer "F.Cu")
+	(via
+		(at 78 102)
+		(size 0.55)
+		(drill 0.3)
+		(layers "F.Cu" "B.Cu")
 		(net "/CORE_CM5/CM5_USB3_RX_P")
 	)
 	(via
 		(at 158 152.6)
-		(size 0.55)
-		(drill 0.3)
-		(layers "F.Cu" "B.Cu")
-		(net "/CORE_CM5/CM5_USB3_RX_P")
-	)
-	(via
-		(at 78 102)
 		(size 0.55)
 		(drill 0.3)
@@
 	)
 	(segment
+		(start 70.04 106.3)
+		(end 82 104)
+		(width 0.2)
+		(layer "F.Cu")
+		(net "/CORE_CM5/CM5_USB3_TX_N")
+	)
+	(segment
+		(start 160 151.2)
+		(end 163.5 151.2)
+		(width 0.2)
+		(layer "F.Cu")
+		(net "/CORE_CM5/CM5_USB3_TX_N")
+	)
+	(segment
 		(start 82 104)
 		(end 160 151.2)
@@
 		(net "/CORE_CM5/CM5_USB3_TX_N")
 	)
-	(segment
-		(start 70.04 106.3)
-		(end 82 104)
-		(width 0.2)
-		(layer "F.Cu")
-		(net "/CORE_CM5/CM5_USB3_TX_N")
-	)
-	(segment
-		(start 160 151.2)
-		(end 163.5 151.2)
-		(width 0.2)
-		(layer "F.Cu")
-		(net "/CORE_CM5/CM5_USB3_TX_N")
-	)
 	(via
 		(at 160 151.2)
@@
 		(layers "F.Cu" "B.Cu")
 		(net "/CORE_CM5/CM5_USB3_TX_N")
+	)
+	(segment
+		(start 162 150.8)
+		(end 163.5 150.8)
+		(width 0.2)
+		(layer "F.Cu")
+		(net "/CORE_CM5/CM5_USB3_TX_P")
 	)
 	(segment
@@
 		(net "/CORE_CM5/CM5_USB3_TX_P")
 	)
-	(segment
-		(start 162 150.8)
-		(end 163.5 150.8)
-		(width 0.2)
-		(layer "F.Cu")
-		(net "/CORE_CM5/CM5_USB3_TX_P")
-	)
 	(via
 		(at 86 106)
@@
 	)
 	(segment
+		(start 151 170)
+		(end 180 170)
+		(width 0.2)
+		(layer "F.Cu")
+		(net "USB_TXN1")
+	)
+	(segment
+		(start 180 170)
+		(end 189.5 170)
+		(width 0.2)
+		(layer "F.Cu")
+		(net "USB_TXN1")
+	)
+	(segment
 		(start 151 153.6)
 		(end 151 170)
@@
 	)
 	(segment
-		(start 151 170)
-		(end 180 170)
-		(width 0.2)
-		(layer "F.Cu")
-		(net "USB_TXN1")
-	)
-	(segment
-		(start 180 170)
-		(end 189.5 170)
-		(width 0.2)
-		(layer "F.Cu")
-		(net "USB_TXN1")
-	)
-	(segment
 		(start 166.5 152.8)
 		(end 235 152.8)
@@
 	)
 	(segment
+		(start 149.4 158)
+		(end 150 170)
+		(width 0.2)
+		(layer "F.Cu")
+		(net "USB_RXP1")
+	)
+	(segment
 		(start 149.4 153.6)
 		(end 149.4 158)
@@
 		(net "USB_RXP1")
 	)
-	(segment
-		(start 149.4 158)
-		(end 150 170)
-		(width 0.2)
-		(layer "F.Cu")
+	(via
+		(at 235 152.8)
+		(size 0.55)
+		(drill 0.3)
+		(layers "F.Cu" "B.Cu")
 		(net "USB_RXP1")
 	)
@@
 		(net "USB_RXP1")
 	)
-	(via
-		(at 235 152.8)
-		(size 0.55)
-		(drill 0.3)
-		(layers "F.Cu" "B.Cu")
+	(segment
+		(start 150 170)
+		(end 140 170)
+		(width 0.2)
+		(layer "B.Cu")
 		(net "USB_RXP1")
 	)
@@
 	)
 	(segment
-		(start 150 170)
-		(end 140 170)
-		(width 0.2)
-		(layer "B.Cu")
-		(net "USB_RXP1")
-	)
-	(segment
 		(start 140 170)
 		(end 140 190)
@@
 	)
 	(via
+		(at 149 200)
+		(size 0.55)
+		(drill 0.3)
+		(layers "F.Cu" "B.Cu")
+		(net "USB_RXN1")
+	)
+	(via
 		(at 240 153.2)
 		(size 0.55)
@@
 		(net "USB_RXN1")
 	)
-	(via
-		(at 149 200)
-		(size 0.55)
-		(drill 0.3)
-		(layers "F.Cu" "B.Cu")
+	(segment
+		(start 240 200)
+		(end 240 153.2)
+		(width 0.2)
+		(layer "B.Cu")
+		(net "USB_RXN1")
+	)
+	(segment
+		(start 250 200)
+		(end 240 200)
+		(width 0.2)
+		(layer "B.Cu")
 		(net "USB_RXN1")
 	)
@@
 	)
 	(segment
-		(start 250 200)
-		(end 240 200)
-		(width 0.2)
-		(layer "B.Cu")
-		(net "USB_RXN1")
-	)
-	(segment
-		(start 240 200)
-		(end 240 153.2)
-		(width 0.2)
-		(layer "B.Cu")
-		(net "USB_RXN1")
-	)
-	(segment
 		(start 190.5 165)
 		(end 192 165)
@@
 	(segment
 		(start 166.5 152)
-		(end 215 152)
+		(end 172 152)
 		(width 0.2)
 		(layer "F.Cu")
@@
 	)
 	(via
-		(at 215 152)
-		(size 0.55)
-		(drill 0.3)
-		(layers "F.Cu" "B.Cu")
-		(net "JMS_USB3_TXP")
-	)
-	(segment
-		(start 215 165)
-		(end 215 152)
-		(width 0.2)
-		(layer "B.Cu")
+		(at 172 152)
+		(size 0.55)
+		(drill 0.3)
+		(layers "F.Cu" "B.Cu")
 		(net "JMS_USB3_TXP")
 	)
 	(segment
 		(start 192 165)
-		(end 215 165)
+		(end 172 165)
+		(width 0.2)
+		(layer "B.Cu")
+		(net "JMS_USB3_TXP")
+	)
+	(segment
+		(start 172 165)
+		(end 172 152)
 		(width 0.2)
 		(layer "B.Cu")
@@
 	(segment
 		(start 166.5 152.4)
-		(end 220 152.4)
+		(end 170 152.4)
 		(width 0.2)
 		(layer "F.Cu")
@@
 	)
 	(via
-		(at 220 152.4)
-		(size 0.55)
-		(drill 0.3)
-		(layers "F.Cu" "B.Cu")
-		(net "JMS_USB3_TXN")
-	)
-	(via
 		(at 194 170)
 		(size 0.55)
@@
 		(net "JMS_USB3_TXN")
 	)
+	(via
+		(at 170 152.4)
+		(size 0.55)
+		(drill 0.3)
+		(layers "F.Cu" "B.Cu")
+		(net "JMS_USB3_TXN")
+	)
 	(segment
 		(start 194 170)
-		(end 220 170)
-		(width 0.2)
-		(layer "B.Cu")
-		(net "JMS_USB3_TXN")
-	)
-	(segment
-		(start 220 170)
-		(end 220 152.4)
-		(width 0.2)
-		(layer "B.Cu")
+		(end 170 170)
+		(width 0.2)
+		(layer "B.Cu")
+		(net "JMS_USB3_TXN")
+	)
+	(segment
+		(start 170 170)
+		(end 170 152.4)
+		(width 0.2)
+		(layer "B.Cu")
