File: pisxme/reva-clean/PHASE24_RTL9210B_LOCAL_OSCILLATOR_V2.kicad_pcb (KiCad board)
At the start: 6 copper layers, 80 x 45 mm, 20 parts, among them J1 M.2 Socket 3 M-key 2280, U1 RTL9210B-CG, U2 W25Q128_SPI_FLASH, Y1 XTAL_25MHz

Commit message: phase24 correct RTL9210B fixture layers
Routing:
- net XTAL_IN: track 0.00 -> 17.3 mm
- net XTAL_OUT: track 0.00 -> 15.7 mm, vias 0 -> 3
- net RSET: track 0.00 -> 12.9 mm, vias 0 -> 2
