File: pisxme/reva-clean/PHASE24_RTL9210B_SUPPORT_BRANCH_RELOCATED_V1.kicad_pcb (KiCad board)
At the start: 6 copper layers, 80 x 45 mm, 20 parts, among them J1 M.2 Socket 3 M-key 2280, U1 RTL9210B-CG, U2 W25Q128_SPI_FLASH, Y1 XTAL_25MHz

Commit message: phase24 stabilize Path B support relocation baseline
Routing:
- net PEDET: track 142.6 -> 0.00 mm, vias 3 -> 0
- net RTL_3V3: track 141.6 -> 0.00 mm, vias 2 -> 0
- net RTL_1V1: track 133.2 -> 0.00 mm, vias 8 -> 0
- net CLKREQ_N: track 103.3 -> 0.00 mm, vias 3 -> 0
- net RTL_5V: track 86.0 -> 0.00 mm, vias 4 -> 0
- net SPISI: track 52.4 -> 0.00 mm
- net SPICLK: track 38.0 -> 0.00 mm, vias 2 -> 0
- net SPISO3: track 35.6 -> 0.00 mm, vias 2 -> 0
- net SPICS: track 31.6 -> 0.00 mm, vias 2 -> 0
- net SPISO: track 31.2 -> 0.00 mm, vias 2 -> 0
