File: pisxme/reva-clean/PHASE24_JMS583_SUPPORT_COHORT_REXT_V6.kicad_pcb (KiCad board)
At the start: 6 copper layers, 300 x 180 mm, 119 parts, among them J1 74221-101LF, J2 A70-112-331N126, J3 1-2199230-4, J4 Amphenol 10171746-00021LF USB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, J6 0039300020, J7 Raspberry-Pi-5-Compute-Module, Q1 CSD19536KCS, Q2 CSD19536KCS, U1 LM74700QDBVRQ1, U2 LM74700QDBVRQ1, U3 TPSM63606RDLR, U4 TPSM63606RDLR, U5 TPSM63606RDLR, U6 TPD4EUSB30, U7 TUSB9261IPVP, U8 Texas_DRT_3, U9 TPD4EUSB30, Y10 25MHz

Commit message: phase24 record post-reconciliation REXT trials
Parts:
- moved R80 8.60 mm to (155.0, 145.0)
Routing:
- net JMS_REXT: track 19.2 -> 20.2 mm
Changed lines of the file:
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@@
 	(footprint "R_0402_1005Metric"
 		(layer "F.Cu")
-		(at 148 140)
+		(at 155 145)
 		(descr "IPC-7351 nominal 0402 resistor; 1.00 x 0.50 mm body; clean-project commodity passive")
 		(property "Reference" "R80"
@@
 	(segment
 		(start 151 135.6)
-		(end 151 142)
+		(end 151 145)
 		(width 0.2)
 		(layer "F.Cu")
@@
 	)
 	(segment
-		(start 147.5 142)
-		(end 147.5 140)
-		(width 0.2)
-		(layer "F.Cu")
-		(net "JMS_REXT")
-	)
-	(segment
-		(start 151 142)
-		(end 147.5 142)
+		(start 151 145)
+		(end 154.5 145)
 		(width 0.2)
 		(layer "F.Cu")
