File: pisxme/reva-clean/PHASE24_JMS583_SUPPORT_COHORT_PROBE.kicad_pcb (KiCad board)
At the start: 6 copper layers, 300 x 180 mm, 119 parts, among them J1 74221-101LF, J2 A70-112-331N126, J3 1-2199230-4, J4 Amphenol 10171746-00021LF USB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, J6 0039300020, J7 Raspberry-Pi-5-Compute-Module, Q1 CSD19536KCS, Q2 CSD19536KCS, U1 LM74700QDBVRQ1, U2 LM74700QDBVRQ1, U3 TPSM63606RDLR, U4 TPSM63606RDLR, U5 TPSM63606RDLR, U6 TPD4EUSB30, U7 TUSB9261IPVP, U8 Texas_DRT_3, U9 TPD4EUSB30, Y10 25MHz

Commit message: phase24 reconcile JMS583 QFN land pattern
Routing:
- net JMS_XAVDDH: track 31.6 -> 34.4 mm

Commit message: phase24 promote JMS REXT placement
Parts:
- moved R80 17.7 mm to (148.0, 130.0)
Changed lines of the file:
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@@
 	(footprint "R_0402_1005Metric"
 		(layer "F.Cu")
-		(at 131 125)
+		(at 148 130)
 		(descr "IPC-7351 nominal 0402 resistor; 1.00 x 0.50 mm body; clean-project commodity passive")
 		(property "Reference" "R80"
@@
 	)
 	(segment
-		(start 136.35 132)
-		(end 133 132)
+		(start 134.85 125)
+		(end 133 125)
 		(width 0.2)
 		(layer "F.Cu")
@@
 	)
 	(segment
-		(start 133 132)
-		(end 133 125)
+		(start 136.35 132)
+		(end 133 132)
 		(width 0.2)
 		(layer "F.Cu")
@@
 	)
 	(segment
-		(start 134.85 125)
+		(start 133 132)
 		(end 133 125)
 		(width 0.2)
@@
 	)
 	(segment
-		(start 136.35 132.4)
-		(end 131 132.4)
+		(start 131 132.4)
+		(end 131 142)
 		(width 0.2)
 		(layer "F.Cu")
@@
 	)
 	(segment
-		(start 118 142)
-		(end 118 147)
+		(start 136.35 132.4)
+		(end 131 132.4)
 		(width 0.2)
 		(layer "F.Cu")
@@
 	)
 	(segment
-		(start 131 132.4)
-		(end 131 142)
+		(start 131 142)
+		(end 118 142)
 		(width 0.2)
 		(layer "F.Cu")
@@
 	)
 	(segment
-		(start 131 142)
-		(end 118 142)
+		(start 118 142)
+		(end 118 147)
 		(width 0.2)
 		(layer "F.Cu")
@@
 	)
 	(segment
-		(start 147 147)
-		(end 147.5 147)
+		(start 136.35 134)
+		(end 134.5 134)
 		(width 0.2)
 		(layer "F.Cu")
@@
 	)
 	(segment
-		(start 147 145)
-		(end 147 147)
+		(start 147 147)
+		(end 147.5 147)
 		(width 0.2)
 		(layer "F.Cu")
@@
 	)
 	(segment
-		(start 136.35 134)
-		(end 134.5 134)
+		(start 147 145)
+		(end 147 147)
 		(width 0.2)
 		(layer "F.Cu")
@@
 	)
 	(via
-		(at 134.5 134)
+		(at 147 145)
 		(size 0.6)
 		(drill 0.3)
@@
 	)
 	(via
-		(at 147 145)
+		(at 134.5 134)
 		(size 0.6)
 		(drill 0.3)
@@
 	)
 	(segment
-		(start 133 143)
-		(end 122 143)
+		(start 122 143)
+		(end 122 145)
 		(width 0.2)
 		(layer "F.Cu")
@@
 	)
 	(segment
-		(start 122 143)
-		(end 122 145)
+		(start 133 143)
+		(end 122 143)
 		(width 0.2)
 		(layer "F.Cu")
@@
 	)
 	(segment
-		(start 142.2 138.6)
-		(end 142.2 140)
+		(start 142.2 140)
+		(end 147 140)
 		(width 0.2)
 		(layer "F.Cu")
@@
 	)
 	(segment
-		(start 147.5 143)
-		(end 147 143)
+		(start 142.2 138.6)
+		(end 142.2 140)
 		(width 0.2)
 		(layer "F.Cu")
@@
 	)
 	(segment
-		(start 142.2 140)
-		(end 147 140)
+		(start 147.5 143)
+		(end 147 143)
 		(width 0.2)
 		(layer "F.Cu")
@@
 	)
 	(segment
-		(start 138.2 130)
-		(end 138.2 140)
+		(start 138.2 140)
+		(end 149 121.5)
 		(width 0.2)
 		(layer "B.Cu")
@@
 	)
 	(segment
-		(start 138.2 140)
-		(end 149 121.5)
+		(start 138.2 130)
+		(end 138.2 140)
 		(width 0.2)
 		(layer "B.Cu")
@@
 	)
 	(segment
-		(start 137.15 125)
+		(start 146 131.4)
 		(end 146 125)
 		(width 0.2)
@@
 	)
 	(segment
-		(start 146 131.4)
+		(start 137.15 125)
 		(end 146 125)
 		(width 0.2)

Commit message: phase24 extend JMS support cohort with AVDDL
Parts:
- moved C83 36.9 mm to (155.0, 147.0)
Routing:
- net JMS_AVDDL: track 0.00 -> 18.1 mm, vias 0 -> 2
Changed lines of the file:
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@@
 	(footprint "C_0402_1005Metric"
 		(layer "F.Cu")
-		(at 137.5 114.5)
+		(at 155 147)
 		(property "Reference" "C83"
 			(at 0 -1.1 0)
@@
 	)
 	(segment
-		(start 134.85 125)
+		(start 133 132)
 		(end 133 125)
 		(width 0.2)
@@
 	)
 	(segment
-		(start 133 132)
+		(start 134.85 125)
 		(end 133 125)
 		(width 0.2)
@@
 	)
 	(segment
-		(start 131 132.4)
-		(end 131 142)
+		(start 119.5 147)
+		(end 118 147)
 		(width 0.2)
 		(layer "F.Cu")
@@
 	)
 	(segment
-		(start 119.5 147)
+		(start 131 142)
+		(end 118 142)
+		(width 0.2)
+		(layer "F.Cu")
+		(net "JMS_VCCK")
+	)
+	(segment
+		(start 118 142)
 		(end 118 147)
 		(width 0.2)
@@
 	)
 	(segment
-		(start 131 142)
-		(end 118 142)
+		(start 131 132.4)
+		(end 131 142)
 		(width 0.2)
 		(layer "F.Cu")
@@
 	)
 	(segment
-		(start 118 142)
-		(end 118 147)
+		(start 147 145)
+		(end 147 147)
 		(width 0.2)
 		(layer "F.Cu")
-		(net "JMS_VCCK")
+		(net "JMS_VCCO")
 	)
 	(segment
@@
 		(net "JMS_VCCO")
 	)
-	(segment
-		(start 147 145)
-		(end 147 147)
-		(width 0.2)
-		(layer "F.Cu")
-		(net "JMS_VCCO")
-	)
 	(via
-		(at 147 145)
+		(at 134.5 134)
 		(size 0.6)
 		(drill 0.3)
@@
 	)
 	(via
-		(at 134.5 134)
+		(at 147 145)
 		(size 0.6)
 		(drill 0.3)
@@
 	)
 	(segment
-		(start 122 143)
-		(end 122 145)
+		(start 136.35 137.6)
+		(end 133 137.6)
 		(width 0.2)
 		(layer "F.Cu")
@@
 	)
 	(segment
-		(start 124.5 145)
-		(end 122 145)
+		(start 133 143)
+		(end 122 143)
 		(width 0.2)
 		(layer "F.Cu")
@@
 	)
 	(segment
-		(start 136.35 137.6)
-		(end 133 137.6)
+		(start 124.5 145)
+		(end 122 145)
 		(width 0.2)
 		(layer "F.Cu")
@@
 	)
 	(segment
-		(start 133 143)
-		(end 122 143)
+		(start 122 143)
+		(end 122 145)
 		(width 0.2)
 		(layer "F.Cu")
@@
 	)
 	(segment
-		(start 147 140)
+		(start 147.5 143)
 		(end 147 143)
 		(width 0.2)
@@
 	)
 	(segment
-		(start 147.5 143)
+		(start 147 140)
 		(end 147 143)
 		(width 0.2)
@@
 	)
 	(segment
-		(start 138.2 131.4)
-		(end 138.2 130)
+		(start 154.5 144)
+		(end 154.5 147)
 		(width 0.2)
 		(layer "F.Cu")
-		(net "JMS_XAVDDH")
+		(net "JMS_AVDDL")
+	)
+	(segment
+		(start 141.8 138.6)
+		(end 141.8 140.5)
+		(width 0.2)
+		(layer "F.Cu")
+		(net "JMS_AVDDL")
+	)
+	(segment
+		(start 154.5 147)
+		(end 154.5 147)
+		(width 0.2)
+		(layer "F.Cu")
+		(net "JMS_AVDDL")
+	)
+	(via
+		(at 154.5 144)
+		(size 0.6)
+		(drill 0.3)
+		(layers "F.Cu" "B.Cu")
+		(net "JMS_AVDDL")
+	)
+	(via
+		(at 141.8 140.5)
+		(size 0.6)
+		(drill 0.3)
+		(layers "F.Cu" "B.Cu")
+		(net "JMS_AVDDL")
+	)
+	(segment
+		(start 141.8 140.5)
+		(end 154.5 144)
+		(width 0.2)
+		(layer "B.Cu")
+		(net "JMS_AVDDL")
 	)
 	(segment
@@
 		(net "JMS_XAVDDH")
 	)
+	(segment
+		(start 138.2 131.4)
+		(end 138.2 130)
+		(width 0.2)
+		(layer "F.Cu")
+		(net "JMS_XAVDDH")
+	)
 	(via
-		(at 138.2 130)
+		(at 149 121.5)
 		(size 0.6)
 		(drill 0.3)
@@
 	)
 	(via
-		(at 149 121.5)
+		(at 138.2 130)
 		(size 0.6)
 		(drill 0.3)

Commit message: phase24 add JMS reset delay cohort
Parts:
- moved C85 28.2 mm to (130.0, 145.0)
Routing:
- net JMS_RESET_N: track 24.2 -> 31.9 mm
Changed lines of the file:
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@@
 	(footprint "C_0402_1005Metric"
 		(layer "F.Cu")
-		(at 127 117)
+		(at 130 145)
 		(property "Reference" "C85"
 			(at 0 -1.1 0)
@@
 	)
 	(segment
+		(start 134.85 125)
+		(end 133 125)
+		(width 0.2)
+		(layer "F.Cu")
+		(net "JMS_VDDREG_5V")
+	)
+	(segment
 		(start 133 132)
 		(end 133 125)
@@
 	)
 	(segment
-		(start 134.85 125)
-		(end 133 125)
+		(start 131 132.4)
+		(end 131 142)
 		(width 0.2)
 		(layer "F.Cu")
-		(net "JMS_VDDREG_5V")
+		(net "JMS_VCCK")
 	)
 	(segment
-		(start 119.5 147)
+		(start 118 142)
 		(end 118 147)
 		(width 0.2)
@@
 	)
 	(segment
-		(start 131 142)
-		(end 118 142)
+		(start 136.35 132.4)
+		(end 131 132.4)
 		(width 0.2)
 		(layer "F.Cu")
@@
 	)
 	(segment
-		(start 118 142)
+		(start 119.5 147)
 		(end 118 147)
 		(width 0.2)
@@
 	)
 	(segment
-		(start 136.35 132.4)
-		(end 131 132.4)
+		(start 131 142)
+		(end 118 142)
 		(width 0.2)
 		(layer "F.Cu")
@@
 	)
 	(segment
-		(start 131 132.4)
-		(end 131 142)
+		(start 147 147)
+		(end 147.5 147)
 		(width 0.2)
 		(layer "F.Cu")
-		(net "JMS_VCCK")
+		(net "JMS_VCCO")
 	)
 	(segment
@@
 		(net "JMS_VCCO")
 	)
-	(segment
-		(start 147 147)
-		(end 147.5 147)
-		(width 0.2)
-		(layer "F.Cu")
-		(net "JMS_VCCO")
-	)
 	(via
 		(at 134.5 134)
@@
 	)
 	(segment
-		(start 134.5 145)
-		(end 147 145)
+		(start 134.5 134)
+		(end 134.5 145)
 		(width 0.2)
 		(layer "B.Cu")
@@
 	)
 	(segment
-		(start 134.5 134)
-		(end 134.5 145)
+		(start 134.5 145)
+		(end 147 145)
 		(width 0.2)
 		(layer "B.Cu")
@@
 	)
 	(segment
-		(start 136.35 137.6)
-		(end 133 137.6)
+		(start 129.5 145)
+		(end 129.5 145)
+		(width 0.2)
+		(layer "F.Cu")
+		(net "JMS_RESET_N")
+	)
+	(segment
+		(start 124 146)
+		(end 129.5 146)
+		(width 0.2)
+		(layer "F.Cu")
+		(net "JMS_RESET_N")
+	)
+	(segment
+		(start 129.5 146)
+		(end 129.5 145)
 		(width 0.2)
 		(layer "F.Cu")
@@
 	(segment
 		(start 124.5 145)
-		(end 122 145)
+		(end 124 146)
 		(width 0.2)
 		(layer "F.Cu")
@@
 	)
 	(segment
+		(start 136.35 137.6)
+		(end 133 137.6)
+		(width 0.2)
+		(layer "F.Cu")
+		(net "JMS_RESET_N")
+	)
+	(segment
 		(start 122 143)
 		(end 122 145)
@@
 	)
 	(segment
-		(start 142.2 140)
-		(end 147 140)
+		(start 124.5 145)
+		(end 122 145)
+		(width 0.2)
+		(layer "F.Cu")
+		(net "JMS_RESET_N")
+	)
+	(segment
+		(start 147 140)
+		(end 147 143)
 		(width 0.2)
 		(layer "F.Cu")
@@
 	)
 	(segment
-		(start 147.5 143)
-		(end 147 143)
+		(start 142.2 140)
+		(end 147 140)
 		(width 0.2)
 		(layer "F.Cu")
@@
 	)
 	(segment
-		(start 147 140)
+		(start 147.5 143)
 		(end 147 143)
 		(width 0.2)
@@
 	)
 	(segment
-		(start 154.5 144)
+		(start 154.5 147)
 		(end 154.5 147)
 		(width 0.2)
@@
 	)
 	(segment
-		(start 141.8 138.6)
-		(end 141.8 140.5)
+		(start 154.5 144)
+		(end 154.5 147)
 		(width 0.2)
 		(layer "F.Cu")
@@
 	)
 	(segment
-		(start 154.5 147)
-		(end 154.5 147)
+		(start 141.8 138.6)
+		(end 141.8 140.5)
 		(width 0.2)
 		(layer "F.Cu")
@@
 	)
 	(via
-		(at 154.5 144)
+		(at 141.8 140.5)
 		(size 0.6)
 		(drill 0.3)
@@
 	)
 	(via
-		(at 141.8 140.5)
+		(at 154.5 144)
 		(size 0.6)
 		(drill 0.3)
@@
 	)
 	(via
-		(at 149 121.5)
+		(at 138.2 130)
 		(size 0.6)
 		(drill 0.3)
@@
 	)
 	(via
-		(at 138.2 130)
+		(at 149 121.5)
 		(size 0.6)
 		(drill 0.3)
@@
 	)
 	(segment
-		(start 146 131.4)
+		(start 137.15 125)
 		(end 146 125)
 		(width 0.2)
@@
 	)
 	(segment
-		(start 137.15 125)
-		(end 146 125)
+		(start 143 131.4)
+		(end 146 131.4)
 		(width 0.2)
 		(layer "F.Cu")
@@
 	)
 	(segment
-		(start 143 131.4)
-		(end 146 131.4)
+		(start 146 131.4)
+		(end 146 125)
 		(width 0.2)
 		(layer "F.Cu")
