File: pisxme/reva-clean/PHASE24_JMS583_SUPPORT_COHORT_V7_NEGATIVE.kicad_pcb (KiCad board)
At the start: 6 copper layers, 300 x 180 mm, 119 parts, among them J1 74221-101LF, J2 A70-112-331N126, J3 1-2199230-4, J4 Amphenol 10171746-00021LF USB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, J6 0039300020, J7 Raspberry-Pi-5-Compute-Module, Q1 CSD19536KCS, Q2 CSD19536KCS, U1 LM74700QDBVRQ1, U2 LM74700QDBVRQ1, U3 TPSM63606RDLR, U4 TPSM63606RDLR, U5 TPSM63606RDLR, U6 TPD4EUSB30, U7 TUSB9261IPVP, U8 Texas_DRT_3, U9 TPD4EUSB30, Y10 25MHz

Commit message: phase24 validate seven-net JMS support cohort
Routing:
- net JMS_VCCK: track 34.4 -> 0.00 mm
- net JMS_XAVDDH: track 31.6 -> 0.00 mm, vias 2 -> 0
- net JMS_VCCO: track 27.8 -> 0.00 mm, vias 2 -> 0
- net JMS_RESET_N: track 24.2 -> 0.00 mm
- net LXO: track 18.2 -> 0.00 mm
- net JMS_VDDREG_5V: track 12.2 -> 0.00 mm
- net JMS_AVDD33: track 9.70 -> 0.00 mm
Changed lines of the file:
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@@
 		(net "/CORE_CM5/CM5_PET0_N")
-	)
-	(segment
-		(start 134.85 125)
-		(end 133 125)
-		(width 0.2)
-		(layer "F.Cu")
-		(net "JMS_VDDREG_5V")
-	)
-	(segment
-		(start 136.35 132)
-		(end 133 132)
-		(width 0.2)
-		(layer "F.Cu")
-		(net "JMS_VDDREG_5V")
-	)
-	(segment
-		(start 133 132)
-		(end 133 125)
-		(width 0.2)
-		(layer "F.Cu")
-		(net "JMS_VDDREG_5V")
-	)
-	(segment
-		(start 136.35 132.4)
-		(end 131 132.4)
-		(width 0.2)
-		(layer "F.Cu")
-		(net "JMS_VCCK")
-	)
-	(segment
-		(start 118 142)
-		(end 118 147)
-		(width 0.2)
-		(layer "F.Cu")
-		(net "JMS_VCCK")
-	)
-	(segment
-		(start 131 142)
-		(end 118 142)
-		(width 0.2)
-		(layer "F.Cu")
-		(net "JMS_VCCK")
-	)
-	(segment
-		(start 131 132.4)
-		(end 131 142)
-		(width 0.2)
-		(layer "F.Cu")
-		(net "JMS_VCCK")
-	)
-	(segment
-		(start 119.5 147)
-		(end 118 147)
-		(width 0.2)
-		(layer "F.Cu")
-		(net "JMS_VCCK")
-	)
-	(segment
-		(start 147 147)
-		(end 147.5 147)
-		(width 0.2)
-		(layer "F.Cu")
-		(net "JMS_VCCO")
-	)
-	(segment
-		(start 136.35 134)
-		(end 134.5 134)
-		(width 0.2)
-		(layer "F.Cu")
-		(net "JMS_VCCO")
-	)
-	(segment
-		(start 147 145)
-		(end 147 147)
-		(width 0.2)
-		(layer "F.Cu")
-		(net "JMS_VCCO")
-	)
-	(via
-		(at 134.5 134)
-		(size 0.6)
-		(drill 0.3)
-		(layers "F.Cu" "B.Cu")
-		(net "JMS_VCCO")
-	)
-	(via
-		(at 147 145)
-		(size 0.6)
-		(drill 0.3)
-		(layers "F.Cu" "B.Cu")
-		(net "JMS_VCCO")
-	)
-	(segment
-		(start 134.5 134)
-		(end 134.5 145)
-		(width 0.2)
-		(layer "B.Cu")
-		(net "JMS_VCCO")
-	)
-	(segment
-		(start 134.5 145)
-		(end 147 145)
-		(width 0.2)
-		(layer "B.Cu")
-		(net "JMS_VCCO")
-	)
-	(segment
-		(start 122 143)
-		(end 122 145)
-		(width 0.2)
-		(layer "F.Cu")
-		(net "JMS_RESET_N")
-	)
-	(segment
-		(start 136.35 137.6)
-		(end 133 137.6)
-		(width 0.2)
-		(layer "F.Cu")
-		(net "JMS_RESET_N")
-	)
-	(segment
-		(start 133 143)
-		(end 122 143)
-		(width 0.2)
-		(layer "F.Cu")
-		(net "JMS_RESET_N")
-	)
-	(segment
-		(start 124.5 145)
-		(end 122 145)
-		(width 0.2)
-		(layer "F.Cu")
-		(net "JMS_RESET_N")
-	)
-	(segment
-		(start 133 137.6)
-		(end 133 143)
-		(width 0.2)
-		(layer "F.Cu")
-		(net "JMS_RESET_N")
-	)
-	(segment
-		(start 142.2 140)
-		(end 147 140)
-		(width 0.2)
-		(layer "F.Cu")
-		(net "JMS_AVDD33")
-	)
-	(segment
-		(start 147 140)
-		(end 147 143)
-		(width 0.2)
-		(layer "F.Cu")
-		(net "JMS_AVDD33")
-	)
-	(segment
-		(start 142.2 138.6)
-		(end 142.2 140)
-		(width 0.2)
-		(layer "F.Cu")
-		(net "JMS_AVDD33")
-	)
-	(segment
-		(start 147.5 143)
-		(end 147 143)
-		(width 0.2)
-		(layer "F.Cu")
-		(net "JMS_AVDD33")
-	)
-	(segment
-		(start 138.2 131.4)
-		(end 138.2 136)
-		(width 0.2)
-		(layer "F.Cu")
-		(net "JMS_XAVDDH")
-	)
-	(segment
-		(start 149 121.5)
-		(end 149.5 120)
-		(width 0.2)
-		(layer "F.Cu")
-		(net "JMS_XAVDDH")
-	)
-	(via
-		(at 149 121.5)
-		(size 0.6)
-		(drill 0.3)
-		(layers "F.Cu" "B.Cu")
-		(net "JMS_XAVDDH")
-	)
-	(via
-		(at 138.2 136)
-		(size 0.6)
-		(drill 0.3)
-		(layers "F.Cu" "B.Cu")
-		(net "JMS_XAVDDH")
-	)
-	(segment
-		(start 138.2 140)
-		(end 149 121.5)
-		(width 0.2)
-		(layer "B.Cu")
-		(net "JMS_XAVDDH")
-	)
-	(segment
-		(start 138.2 136)
-		(end 138.2 140)
-		(width 0.2)
-		(layer "B.Cu")
-		(net "JMS_XAVDDH")
-	)
-	(segment
-		(start 146 131.4)
-		(end 146 125)
-		(width 0.2)
-		(layer "F.Cu")
-		(net "LXO")
-	)
-	(segment
-		(start 137.15 125)
-		(end 146 125)
-		(width 0.2)
-		(layer "F.Cu")
-		(net "LXO")
-	)
-	(segment
-		(start 143 131.4)
-		(end 146 131.4)
-		(width 0.2)
-		(layer "F.Cu")
-		(net "LXO")
 	)
 	(zone

Commit message: phase24 promote JMS REXT placement
Parts:
- moved R80 17.7 mm to (148.0, 130.0)
Changed lines of the file:
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@@
 	(footprint "R_0402_1005Metric"
 		(layer "F.Cu")
-		(at 131 125)
+		(at 148 130)
 		(descr "IPC-7351 nominal 0402 resistor; 1.00 x 0.50 mm body; clean-project commodity passive")
 		(property "Reference" "R80"

Commit message: phase24 extend JMS support cohort with AVDDL
Parts:
- moved C83 36.9 mm to (155.0, 147.0)
Changed lines of the file:
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@@
 	(footprint "C_0402_1005Metric"
 		(layer "F.Cu")
-		(at 137.5 114.5)
+		(at 155 147)
 		(property "Reference" "C83"
 			(at 0 -1.1 0)

Commit message: phase24 add JMS reset delay cohort
Parts:
- moved C85 28.2 mm to (130.0, 145.0)
Changed lines of the file:
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@@
 	(footprint "C_0402_1005Metric"
 		(layer "F.Cu")
-		(at 127 117)
+		(at 130 145)
 		(property "Reference" "C85"
 			(at 0 -1.1 0)
