File: pisxme/reva-clean/PHASE24_JMS583_CRYSTAL_ESCAPE_PROBE.kicad_pcb (KiCad board)
At the start: 6 copper layers, 300 x 180 mm, 119 parts, among them J1 74221-101LF, J2 A70-112-331N126, J3 1-2199230-4, J4 Amphenol 10171746-00021LF USB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, J6 0039300020, J7 Raspberry-Pi-5-Compute-Module, Q1 CSD19536KCS, Q2 CSD19536KCS, U1 LM74700QDBVRQ1, U2 LM74700QDBVRQ1, U3 TPSM63606RDLR, U4 TPSM63606RDLR, U5 TPSM63606RDLR, U6 TPD4EUSB30, U7 TUSB9261IPVP, U8 Texas_DRT_3, U9 TPD4EUSB30, Y10 25MHz

Commit message: phase24 recheck JMS crystal fixture
Parts:
- moved R80 17.7 mm to (148.0, 130.0)
Changed lines of the file:
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@@
 	(footprint "R_0402_1005Metric"
 		(layer "F.Cu")
-		(at 131 125)
+		(at 148 130)
 		(descr "IPC-7351 nominal 0402 resistor; 1.00 x 0.50 mm body; clean-project commodity passive")
 		(property "Reference" "R80"
@@
 		(layer "F.Cu")
 		(at 140 135)
-		(descr "JMS583_QFN64_8x8; TI RUA0042A, 9.0 x 3.5 mm WQFN")
+		(descr "JMS583_QFN64_8x8; JMicron JMS583 QFN64 8 x 8 mm; datasheet Rev 2.1 Figure 4")
 		(property "Reference" "U11"
 			(at 0 -5.4 0)
@@
 		(duplicate_pad_numbers_are_jumpers no)
 		(fp_rect
-			(start -2.1 -4.6)
-			(end 2.1 4.6)
+			(start -4.6 -4.6)
+			(end 4.6 4.6)
 			(stroke
 				(width 0.05)
@@
 			(pintype "passive")
 		)
+		(pad "65" smd roundrect
+			(at 0 0)
+			(size 0.7 0.2)
+			(layers "F.Cu" "F.Mask" "F.Paste")
+			(roundrect_rratio 0.05)
+			(net "POWER_GND")
+			(pinfunction "POWER_GND")
+			(pintype "passive")
+		)
 		(embedded_fonts no)
 	)
@@
 	)
 	(segment
-		(start 137.4 131.4)
-		(end 137.4 129)
+		(start 137.4 129)
+		(end 134 129)
 		(width 0.15)
 		(layer "F.Cu")
@@
 	)
 	(segment
-		(start 137.4 129)
-		(end 134 129)
+		(start 137.4 131.4)
+		(end 137.4 129)
 		(width 0.15)
 		(layer "F.Cu")
@@
 	)
 	(via
-		(at 134 129)
+		(at 147 122)
 		(size 0.5)
 		(drill 0.3)
@@
 	)
 	(via
-		(at 147 122)
+		(at 134 129)
 		(size 0.5)
 		(drill 0.3)
@@
 	)
 	(segment
-		(start 134 129)
-		(end 147 129)
+		(start 147 129)
+		(end 147 122)
 		(width 0.15)
 		(layer "B.Cu")
@@
 	)
 	(segment
-		(start 147 129)
-		(end 147 122)
+		(start 134 129)
+		(end 147 129)
 		(width 0.15)
 		(layer "B.Cu")
@@
 	)
 	(segment
-		(start 137.8 128)
-		(end 140 128)
+		(start 137.8 131.4)
+		(end 137.8 128)
 		(width 0.15)
 		(layer "F.Cu")
@@
 	)
 	(segment
-		(start 137.8 131.4)
-		(end 137.8 128)
+		(start 137.8 128)
+		(end 140 128)
 		(width 0.15)
 		(layer "F.Cu")
@@
 	)
 	(via
-		(at 140 128)
+		(at 146 123)
 		(size 0.5)
 		(drill 0.3)
@@
 	)
 	(via
-		(at 146 123)
+		(at 140 128)
 		(size 0.5)
 		(drill 0.3)
