File: pisxme/reva-clean/PHASE24_RTL9210B_STAGGERED_SOURCE_CLEANFIELD_V1149.kicad_pcb (KiCad board)
At the start: 6 copper layers, 80 x 45 mm, 12 parts, among them J1 M.2 Socket 3 M-key 2280, U1 RTL9210B-CG, U2 W25Q128_SPI_FLASH, Y1 XTAL_25MHz

Commit message: phase24: assert native branch pruning
Routing:
- net RTL_3V3: track 135.1 -> 131.1 mm, vias 10 -> 9
Changed lines of the file:
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@@
+	)
+	(segment
+		(start 94.05 68)
+		(end 95 68)
+		(width 0.2)
+		(layer "F.Cu")
+		(net "RTL_1V1")
 	)
 	(segment
@@
 	)
 	(segment
-		(start 94.05 68)
-		(end 95 68)
-		(width 0.2)
-		(layer "F.Cu")
-		(net "RTL_1V1")
-	)
-	(segment
 		(start 100.8 73.95)
 		(end 100.8 75)
@@
 	)
 	(via
+		(at 95 68)
+		(size 0.6)
+		(drill 0.3)
+		(layers "F.Cu" "B.Cu")
+		(net "RTL_1V1")
+	)
+	(via
 		(at 122.8 51)
 		(size 0.6)
@@
 	(via
 		(at 102.5 75)
-		(size 0.6)
-		(drill 0.3)
-		(layers "F.Cu" "B.Cu")
-		(net "RTL_1V1")
-	)
-	(via
-		(at 95 68)
 		(size 0.6)
 		(drill 0.3)
@@
 	)
 	(segment
+		(start 92.8 70)
+		(end 92.8 75)
+		(width 0.2)
+		(layer "B.Cu")
+		(net "RTL_1V1")
+	)
+	(segment
+		(start 112 52)
+		(end 122.8 52)
+		(width 0.2)
+		(layer "B.Cu")
+		(net "RTL_1V1")
+	)
+	(segment
+		(start 92.8 75)
+		(end 102.5 75)
+		(width 0.2)
+		(layer "B.Cu")
+		(net "RTL_1V1")
+	)
+	(segment
+		(start 102.5 64.8)
+		(end 102 64.8)
+		(width 0.2)
+		(layer "B.Cu")
+		(net "RTL_1V1")
+	)
+	(segment
 		(start 95 68)
 		(end 95 75)
@@
 	)
 	(segment
-		(start 92.8 70)
-		(end 92.8 75)
-		(width 0.2)
-		(layer "B.Cu")
-		(net "RTL_1V1")
-	)
-	(segment
-		(start 112 52)
-		(end 122.8 52)
-		(width 0.2)
-		(layer "B.Cu")
-		(net "RTL_1V1")
-	)
-	(segment
 		(start 92.8 75)
 		(end 102.5 75)
@@
 	)
 	(segment
-		(start 102.5 64.8)
-		(end 102 64.8)
+		(start 95 75)
+		(end 102.5 75)
 		(width 0.2)
 		(layer "B.Cu")
@@
 	)
 	(segment
-		(start 92.8 75)
-		(end 102.5 75)
-		(width 0.2)
-		(layer "B.Cu")
-		(net "RTL_1V1")
-	)
-	(segment
 		(start 122.8 52)
 		(end 122.8 51)
@@
 	)
 	(segment
-		(start 95 75)
-		(end 102.5 75)
-		(width 0.2)
-		(layer "B.Cu")
-		(net "RTL_1V1")
-	)
-	(segment
 		(start 102 64.8)
 		(end 97.8 64.8)
@@
 	)
 	(segment
+		(start 92 66.8)
+		(end 92 65)
+		(width 0.2)
+		(layer "F.Cu")
+		(net "RTL_3V3")
+	)
+	(segment
 		(start 101.95 66.8)
 		(end 103 66.8)
@@
 	)
 	(segment
-		(start 92 66.8)
-		(end 92 65)
-		(width 0.2)
-		(layer "F.Cu")
-		(net "RTL_3V3")
-	)
-	(segment
 		(start 121.2 80)
 		(end 121.8 80)
@@
 	)
 	(segment
+		(start 94.05 66.8)
+		(end 92 66.8)
+		(width 0.2)
+		(layer "F.Cu")
+		(net "RTL_3V3")
+	)
+	(segment
 		(start 121.8 80)
 		(end 121.8 78)
@@
 		(net "RTL_3V3")
 	)
-	(segment
-		(start 94.05 66.8)
-		(end 92 66.8)
-		(width 0.2)
-		(layer "F.Cu")
-		(net "RTL_3V3")
-	)
 	(via
 		(at 119.8 78)
@@
 	)
 	(via
+		(at 92 65)
+		(size 0.6)
+		(drill 0.3)
+		(layers "F.Cu" "B.Cu")
+		(net "RTL_3V3")
+	)
+	(via
 		(at 100.9 72.4)
 		(size 0.6)
@@
 	)
 	(via
-		(at 93 66.8)
-		(size 0.6)
-		(drill 0.3)
-		(layers "F.Cu" "B.Cu")
-		(net "RTL_3V3")
-	)
-	(via
 		(at 108 64)
-		(size 0.6)
-		(drill 0.3)
-		(layers "F.Cu" "B.Cu")
-		(net "RTL_3V3")
-	)
-	(via
-		(at 92 65)
 		(size 0.6)
 		(drill 0.3)
@@
 	)
 	(segment
+		(start 100.5 65)
+		(end 100.5 64)
+		(width 0.2)
+		(layer "B.Cu")
+		(net "RTL_3V3")
+	)
+	(segment
 		(start 119.2 51)
 		(end 119.2 51)
@@
 	)
 	(segment
+		(start 123.5 49)
+		(end 119.2 49)
+		(width 0.2)
+		(layer "B.Cu")
+		(net "RTL_3V3")
+	)
+	(segment
 		(start 92 65)
 		(end 100.5 65)
@@
 	)
 	(segment
-		(start 100.9 68.4)
-		(end 100.9 72.4)
-		(width 0.2)
-		(layer "B.Cu")
-		(net "RTL_3V3")
-	)
-	(segment
-		(start 123.5 49)
-		(end 119.2 49)
-		(width 0.2)
-		(layer "B.Cu")
-		(net "RTL_3V3")
-	)
-	(segment
 		(start 108 50)
 		(end 119.2 50)
@@
 	)
 	(segment
-		(start 100.5 65)
-		(end 100.5 64)
-		(width 0.2)
-		(layer "B.Cu")
-		(net "RTL_3V3")
-	)
-	(segment
 		(start 119.8 74)
 		(end 119.8 78)
@@
 	)
 	(segment
+		(start 93 67.2)
+		(end 92 67.2)
+		(width 0.2)
+		(layer "F.Cu")
+		(net "XTAL_IN")
+	)
+	(segment
+		(start 94.05 67.2)
+		(end 93 67.2)
+		(width 0.2)
+		(layer "F.Cu")
+		(net "XTAL_IN")
+	)
+	(segment
 		(start 92 67.2)
 		(end 90.5 66.8)
 		(width 0.2)
 		(layer "F.Cu")
-		(net "XTAL_IN")
-	)
-	(segment
-		(start 94.05 67.2)
-		(end 93 67.2)
-		(width 0.2)
-		(layer "F.Cu")
-		(net "XTAL_IN")
-	)
-	(segment
-		(start 93 67.2)
-		(end 92 67.2)
-		(width 0.2)
-		(layer "F.Cu")
