File: pisxme/reva-clean/PHASE24_RTL9210B_SOURCE_ROW_STAGGERED_FUNNEL.kicad_pcb (KiCad board)
At the start: 6 copper layers, 100.1 x 55.1 mm, 19 parts, among them J1 M.2 Socket 3 M-key 2280, U1 RTL9210B-CG, U2 W25Q128_SPI_FLASH, Y1 XTAL_25MHz

Commit message: phase24: record final source handoff discriminator
Routing:
- net CLKREQ_N: track 67.7 -> 69.5 mm
- net PERST_N: track 31.5 -> 33.0 mm
- net RTL_1V1: track 93.2 -> 94.3 mm
- net RTL_5V: track 72.7 -> 73.6 mm
